Commit message: 

File: description/inertial_macros.xacro (robot description, xacro)
@@ -1,33 +1,32 @@
 <?xml version="1.0"?>
-<robot xmlns:xacro="http://ros.org/wiki/xacro">
-  <!-- Sphere inertia macro -->
-  <xacro:macro name="inertial_sphere" params="mass radius *origin">
-    <inertial>
-      <xacro:insert_block name="origin"/>
-      <mass value="${mass}"/>
-      <inertia ixx="${(2.0/5.0)*mass*(radius*radius)}" ixy="0" ixz="0"
-               iyy="${(2.0/5.0)*mass*(radius*radius)}" iyz="0"
-               izz="${(2.0/5.0)*mass*(radius*radius)}"/>
-    </inertial>
-  </xacro:macro>
-  <!-- Box inertia macro -->
-  <xacro:macro name="inertial_box" params="mass x y z *origin">
-    <inertial>
-      <xacro:insert_block name="origin"/>
-      <mass value="${mass}"/>
-      <inertia ixx="${(1.0/12.0)*mass*(y*y+z*z)}" ixy="0" ixz="0"
-               iyy="${(1.0/12.0)*mass*(x*x+z*z)}" iyz="0"
-               izz="${(1.0/12.0)*mass*(x*x+y*y)}"/>
-    </inertial>
-  </xacro:macro>
-  <!-- Cylinder inertia macro -->
-  <xacro:macro name="inertial_cylinder" params="mass length radius *origin">
-    <inertial>
-      <xacro:insert_block name="origin"/>
-      <mass value="${mass}"/>
-      <inertia ixx="${(1.0/12.0)*mass*(3*radius*radius + length*length)}" ixy="0" ixz="0"
-               iyy="${(1.0/12.0)*mass*(3*radius*radius + length*length)}" iyz="0"
-               izz="${(1.0/2.0)*mass*(radius*radius)}"/>
-    </inertial>
-  </xacro:macro>
+<robot xmlns:xacro="http://www.ros.org/wiki/xacro" >
+    <!-- Specify some standard inertial calculations https://en.wikipedia.org/wiki/List_of_moments_of_inertia -->
+    <!-- These make use of xacro's mathematical functionality -->
+    <xacro:macro name="inertial_sphere" params="mass radius *origin">
+        <inertial>
+            <xacro:insert_block name="origin"/>
+            <mass value="${mass}" />
+            <inertia ixx="${(2/5) * mass * (radius*radius)}" ixy="0.0" ixz="0.0"
+                    iyy="${(2/5) * mass * (radius*radius)}" iyz="0.0"
+                    izz="${(2/5) * mass * (radius*radius)}" />
+        </inertial>
+    </xacro:macro>
+    <xacro:macro name="inertial_box" params="mass x y z *origin">
+        <inertial>
+            <xacro:insert_block name="origin"/>
+            <mass value="${mass}" />
+            <inertia ixx="${(1/12) * mass * (y*y+z*z)}" ixy="0.0" ixz="0.0"
+                    iyy="${(1/12) * mass * (x*x+z*z)}" iyz="0.0"
+                    izz="${(1/12) * mass * (x*x+y*y)}" />
+        </inertial>
+    </xacro:macro>
+    <xacro:macro name="inertial_cylinder" params="mass length radius *origin">
+        <inertial>
+            <xacro:insert_block name="origin"/>
+            <mass value="${mass}" />
+            <inertia ixx="${(1/12) * mass * (3*radius*radius + length*length)}" ixy="0.0" ixz="0.0"
+                    iyy="${(1/12) * mass * (3*radius*radius + length*length)}" iyz="0.0"
+                    izz="${(1/2) * mass * (radius*radius)}" />
+        </inertial>
+    </xacro:macro>
 </robot>

File: description/robot_core.xacro (robot description, xacro)
@@ -1,75 +1,111 @@
 <?xml version="1.0"?>
-<robot xmlns:xacro="http://ros.org/wiki/xacro">
-  <!-- Define constants -->
-  <xacro:property name="pi" value="3.141592653589793"/>
-  <!-- Include macros (adjust package/path if needed) -->
-  <xacro:include filename="inertial_macros.xacro"/>
-  <!-- Materials -->
-  <material name="white"><color rgba="1 1 1 1"/></material>
-  <material name="orange"><color rgba="1 0.3 0.1 1"/></material>
-  <material name="blue"><color rgba="0.2 0.2 1 1"/></material>
-  <material name="black"><color rgba="0 0 0 1"/></material>
-  <!-- Base link -->
-  <link name="base_link"/>
-  <!-- Chassis -->
-  <joint name="chassis_joint" type="fixed">
-    <parent link="base_link"/>
-    <child link="chassis"/>
-    <origin xyz="-0.1 0 0"/>
-  </joint>
-  <link name="chassis">
-    <visual>
-      <origin xyz="0.15 0 0.075"/>
-      <geometry><box size="0.3 0.3 0.15"/></geometry>
-      <material name="white"/>
-    </visual>
-    <collision>
-      <origin xyz="0.15 0 0.075"/>
-      <geometry><box size="0.3 0.3 0.15"/></geometry>
-    </collision>
-    <xacro:inertial_box mass="0.5" x="0.3" y="0.3" z="0.15">
-      <origin xyz="0.15 0 0.075" rpy="0 0 0"/>
-    </xacro:inertial_box>
-  </link>
-  <!-- Left wheel -->
-  <joint name="left_wheel_joint" type="continuous">
-    <parent link="base_link"/>
-    <child link="left_wheel"/>
-    <origin xyz="0 0.175 0" rpy="-${pi/2} 0 0"/>
-    <axis xyz="0 0 1"/>
-  </joint>
-  <link name="left_wheel">
-    <visual><geometry><cylinder radius="0.05" length="0.04"/></geometry><material name="blue"/></visual>
-    <collision><geometry><cylinder radius="0.05" length="0.04"/></geometry></collision>
-    <xacro:inertial_cylinder mass="0.1" length="0.04" radius="0.05">
-      <origin xyz="0 0 0" rpy="0 0 0"/>
-    </xacro:inertial_cylinder>
-  </link>
-  <!-- Right wheel -->
-  <joint name="right_wheel_joint" type="continuous">
-    <parent link="base_link"/>
-    <child link="right_wheel"/>
-    <origin xyz="0 -0.175 0" rpy="${pi/2} 0 0"/>
-    <axis xyz="0 0 -1"/>
-  </joint>
-  <link name="right_wheel">
-    <visual><geometry><cylinder radius="0.05" length="0.04"/></geometry><material name="blue"/></visual>
-    <collision><geometry><cylinder radius="0.05" length="0.04"/></geometry></collision>
-    <xacro:inertial_cylinder mass="0.1" length="0.04" radius="0.05">
-      <origin xyz="0 0 0" rpy="0 0 0"/>
-    </xacro:inertial_cylinder>
-  </link>
-  <!-- Caster wheel -->
-  <joint name="caster_wheel_joint" type="fixed">
-    <parent link="chassis"/>
-    <child link="caster_wheel"/>
-    <origin xyz="0.24 0 0"/>
-  </joint>
-  <link name="caster_wheel">
-    <visual><geometry><sphere radius="0.05"/></geometry><material name="black"/></visual>
-    <collision><geometry><sphere radius="0.05"/></geometry></collision>
-    <xacro:inertial_sphere mass="0.1" radius="0.05">
-      <origin xyz="0 0 0" rpy="0 0 0"/>
-    </xacro:inertial_sphere>
-  </link>
+<robot xmlns:xacro="http://www.ros.org/wiki/xacro" >
+    <xacro:include filename="inertial_macros.xacro"/>
+    <material name="white">
+        <color rgba="1 1 1 1" />
+    </material>
+    <material name="orange">
+        <color rgba="1 0.3 0.1 1"/>
+    </material>
+    <material name="blue">
+        <color rgba="0.2 0.2 1 1"/>
+    </material>
+    <material name="black">
+        <color rgba="0 0 0 1"/>
+    </material>
+    <!-- BASE LINK -->
+    <link name="base_link">
+    </link>
+    <!-- CHASSIS LINK -->
+    <joint name="chassis_joint" type="fixed">
+        <parent link="base_link"/>
+        <child link="chassis"/>
+        <origin xyz="-0.1 0 0"/>
+    </joint>
+    <link name="chassis">
+        <visual>
+            <origin xyz="0.15 0 0.075"/>
+            <geometry>
+                <box size="0.3 0.3 0.15"/>
+            </geometry>
+            <material name="white"/>
+        </visual>
+        <collision>
+            <origin xyz="0.15 0 0.075"/>
+            <geometry>
+                <box size="0.3 0.3 0.15"/>
+            </geometry>
+        </collision>
+        <xacro:inertial_box mass="0.5" x="0.3" y="0.3" z="0.15">
+            <origin xyz="0.15 0 0.075" rpy="0 0 0"/>
+        </xacro:inertial_box>
+    </link>
+    <!-- LEFT WHEEL LINK -->
+    <joint name="left_wheel_joint" type="continuous">
+        <parent link="base_link"/>
+        <child link="left_wheel"/>
+        <origin xyz="0 0.175 0" rpy="-${pi/2} 0 0" />
+        <axis xyz="0 0 1"/>
+    </joint>
+    <link name="left_wheel">
+        <visual>
+            <geometry>
+                <cylinder radius="0.05" length="0.04"/>
+            </geometry>
+            <material name="blue"/>
+        </visual>
+        <collision>
+            <geometry>
+                <cylinder radius="0.05" length="0.04"/>
+            </geometry>
+        </collision>
+        <xacro:inertial_cylinder mass="0.1" length="0.04" radius="0.05">
+            <origin xyz="0 0 0" rpy="0 0 0"/>
+        </xacro:inertial_cylinder>
+    </link>
+    <!-- RIGHT WHEEL LINK -->
+    <joint name="right_wheel_joint" type="continuous">
+        <parent link="base_link"/>
+        <child link="right_wheel"/>
+        <origin xyz="0 -0.175 0" rpy="${pi/2} 0 0" />
+        <axis xyz="0 0 -1"/>
+    </joint>
+    <link name="right_wheel">
+        <visual>
+            <geometry>
+                <cylinder radius="0.05" length="0.04"/>
+            </geometry>
+            <material name="blue"/>
+        </visual>
+        <collision>
+            <geometry>
+                <cylinder radius="0.05" length="0.04"/>
+            </geometry>
+        </collision>
+        <xacro:inertial_cylinder mass="0.1" length="0.04" radius="0.05">
+            <origin xyz="0 0 0" rpy="0 0 0"/>
+        </xacro:inertial_cylinder>
+    </link>
+    <!-- CASTER WHEEL LINK -->
+    <joint name="caster_wheel_joint" type="fixed">
+        <parent link="chassis"/>
+        <child link="caster_wheel"/>
+        <origin xyz="0.24 0 0"/>
+    </joint>
+    <link name="caster_wheel">
+        <visual>
+            <geometry>
+                <sphere radius="0.05"/>
+            </geometry>
+            <material name="black"/>
+        </visual>
+        <collision>
+            <geometry>
+                <sphere radius="0.05"/>
+            </geometry>
+        </collision>
+        <xacro:inertial_sphere mass="0.1" radius="0.05">
+            <origin xyz="0 0 0" rpy="0 0 0"/>
+        </xacro:inertial_sphere>
+    </link>
 </robot>
