Commit message: 

File: description/gazebo_control.xacro (robot description, xacro)
@@ -4,6 +4,6 @@
         <plugin name="gz::sim::systems::DiffDrive" filename="gz-sim-diff-drive-system">
             <!-- Wheel Information -->
-            <left_joint>left_wheel_joint</left_joint>
-            <right_joint>right_wheel_joint</right_joint>
+            <left_joint>joint-chassis-front-left-wheel</left_joint>
+            <right_joint>joint-chassis-front-right-wheel</right_joint>
             <wheel_separation>0.297</wheel_separation>
             <wheel_radius>0.033</wheel_radius>
@@ -23,6 +23,6 @@
             name="gz::sim::systems::JointStatePublisher">
             <topic>joint_states</topic>
-            <joint_name>left_wheel_joint</joint_name>
-            <joint_name>right_wheel_joint</joint_name>
+            <joint_name>joint-chassis-front-left-wheel</joint_name>
+            <joint_name>joint-chassis-front-right-wheel</joint_name>
         </plugin>
     </gazebo>

File: description/gz_ros2_control.xacro (robot description, xacro)
@@ -5,5 +5,5 @@
                 <plugin>gz_ros2_control/GazeboCustomSimSystem</plugin>
             </hardware>
-            <joint name="left_wheel_joint">
+            <joint name="joint-chassis-front-left-wheel">
                 <command_interface name="velocity">
                     <param name="min">-10</param>
@@ -13,5 +13,5 @@
                 <state_interface name="position"/>
             </joint>
-            <joint name="right_wheel_joint">
+            <joint name="joint-chassis-front-right-wheel">
                 <command_interface name="velocity">
                     <param name="min">-10</param>

File: description/robot_core.xacro (robot description, xacro)
@@ -1,158 +1,168 @@
 <?xml version="1.0"?>
 <robot xmlns:xacro="http://www.ros.org/wiki/xacro" >
-    <xacro:include filename="inertial_macros.xacro"/>
-    <material name="white">
-        <color rgba="1 1 1 1" />
-    </material>
-    <material name="orange">
-        <color rgba="1 0.3 0.1 1"/>
-    </material>
-    <material name="blue">
-        <color rgba="0.2 0.2 1 1"/>
-    </material>
-    <material name="black">
-        <color rgba="0 0 0 1"/>
-    </material>
-    <!-- BASE LINK -->
-    <link name="base_link">
-    </link>
-    <!-- CHASSIS LINK -->
-    <joint name="chassis_joint" type="fixed">
-        <parent link="base_link"/>
-        <child link="chassis"/>
-        <origin xyz="-0.1 0 0"/>
-    </joint>
-    <link name="chassis">
-        <visual>
-            <origin xyz="0.15 0 0.075"/>
-            <geometry>
-                <box size="0.3 0.3 0.15"/>
-            </geometry>
-            <material name="white"/>
-        </visual>
-        <collision>
-            <origin xyz="0.15 0 0.075"/>
-            <geometry>
-                <box size="0.3 0.3 0.15"/>
-            </geometry>
-        </collision>
-        <xacro:inertial_box mass="0.5" x="0.3" y="0.3" z="0.15">
-            <origin xyz="0.15 0 0.075" rpy="0 0 0"/>
-        </xacro:inertial_box>
-    </link>
-    <gazebo reference="chassis">
-        <material>Gazebo/White</material>
-    </gazebo>
-    <!-- LEFT WHEEL LINK -->
-    <joint name="left_wheel_joint" type="continuous">
-        <parent link="base_link"/>
-        <child link="left_wheel"/>
-        <origin xyz="0 0.175 0" rpy="-${pi/2} 0 0" />
-        <axis xyz="0 0 1"/>
-    </joint>
-    <link name="left_wheel">
-        <visual>
-            <geometry>
-                <cylinder radius="0.05" length="0.04"/>
-            </geometry>
-            <material name="blue"/>
-        </visual>
-        <collision>
-            <geometry>
-                <cylinder radius="0.05" length="0.04"/>
-            </geometry>
-        </collision>
-        <xacro:inertial_cylinder mass="0.1" length="0.04" radius="0.05">
-            <origin xyz="0 0 0" rpy="0 0 0"/>
-        </xacro:inertial_cylinder>
-        <surface>
-           <contact>
-            <ode/>
-           </contact>
-           <friction>
-             <ode>
-                  <mu>1.0</mu>
-                  <mu2>1.0</mu2>
-             </ode>
-            </friction>
-        </surface>
-    </link>
-    <gazebo reference="left_wheel">
-        <material>Gazebo/Blue</material>
-    </gazebo>
-    <!-- RIGHT WHEEL LINK -->
-    <joint name="right_wheel_joint" type="continuous">
-        <parent link="base_link"/>
-        <child link="right_wheel"/>
-        <origin xyz="0 -0.175 0" rpy="${pi/2} 0 0" />
-        <axis xyz="0 0 -1"/>
-    </joint>
-    <link name="right_wheel">
-        <visual>
-            <geometry>
-                <cylinder radius="0.05" length="0.04"/>
-            </geometry>
-            <material name="blue"/>
-        </visual>
-        <collision>
-            <geometry>
-                <cylinder radius="0.05" length="0.04"/>
-            </geometry>
-        </collision>
-        <xacro:inertial_cylinder mass="0.1" length="0.04" radius="0.05">
-            <origin xyz="0 0 0" rpy="0 0 0"/>
-        </xacro:inertial_cylinder>
-        <surface>
-           <contact>
-            <ode/>
-           </contact>
-           <friction>
-             <ode>
-                  <mu>1.0</mu>
-                  <mu2>1.0</mu2>
-             </ode>
-            </friction>
-        </surface>
-    </link>
-    <gazebo reference="right_wheel">
-        <material>Gazebo/Blue</material>
-    </gazebo>
-    <!-- CASTER WHEEL LINK -->
-    <joint name="caster_wheel_joint" type="fixed">
-        <parent link="chassis"/>
-        <child link="caster_wheel"/>
-        <origin xyz="0.24 0 0"/>
-    </joint>
-    <link name="caster_wheel">
-        <visual>
-            <geometry>
-                <sphere radius="0.05"/>
-            </geometry>
-            <material name="black"/>
-        </visual>
-        <collision>
-            <geometry>
-                <sphere radius="0.05"/>
-            </geometry>
-        </collision>
-        <xacro:inertial_sphere mass="0.1" radius="0.05">
-            <origin xyz="0 0 0" rpy="0 0 0"/>
-        </xacro:inertial_sphere>
-        <surface>
-           <contact>
-            <ode/>
-           </contact>
-           <friction>
-             <ode>
-                  <mu>1.0</mu>
-                  <mu2>1.0</mu2>
-             </ode>
-            </friction>
-        </surface>
-    </link>
-    <gazebo reference="caster_wheel">
-        <material>Gazebo/Black</material>
-        <mu1 value="0.001"/>
-        <mu2 value="0.001"/>
-    </gazebo>
+<robot name="car-robot">
+  <!--dummy link-->
+  <link name="base_link"/>
+  <!--chassis link-->
+  <link name="chassis-link">
+    <visual>
+      <origin rpy="0 0 0" xyz="0 0 0"/>
+      <geometry>
+        <box size="0.14 0.12 0.01"/>
+      </geometry>
+      <material name="brown">
+        <color rgba="0.3 0 0.4 1"/>
+      </material>
+    </visual>
+    <collision>
+      <origin rpy="0 0 0" xyz="0 0 0"/>
+      <geometry>
+        <box size="0.14 0.12 0.01"/>
+      </geometry>
+    </collision>
+    <inertial>
+      <mass value="0.4"/>
+      <inertia ixx="0.00048333" ixy="0" ixz="0" iyy="0.0013367" iyz="0" izz="0.0018133"/>
+    </inertial>
+  </link>
+  <joint name="joint-base-chassis" type="fixed">
+    <parent link="base_link"/>
+    <child link="chassis-link"/>
+    <origin rpy="0 0 0" xyz="0 0 0.02"/>
+  </joint>
+  <material name="blue">
+    <color rgba="0 0.4 0.5 1"/>
+  </material>
+  <!-- ${x_position}-${y_position}-wheel-link -->
+  <link name="front-right-wheel-link">
+    <visual>
+      <origin rpy="1.5707963267948966 0 0" xyz="0 0 0"/>
+      <geometry>
+        <cylinder length="0.01" radius="0.02"/>
+      </geometry>
+      <material name="blue"/>
+    </visual>
+    <collision>
+      <origin rpy="1.5707963267948966 0 0" xyz="0 0 0"/>
+      <geometry>
+        <cylinder length="0.01" radius="0.02"/>
+      </geometry>
+    </collision>
+    <inertial>
+      <origin rpy="1.5707963267948966 0 0" xyz="0 0 0"/>
+      <mass value="0.2"/>
+      <inertia ixx="2.166666666666667e-05" ixy="0" ixz="0" iyy="2.166666666666667e-05" iyz="0" izz="4e-05"/>
+    </inertial>
+  </link>
+  <joint name="joint-chassis-front-right-wheel" type="continuous">
+    <parent link="chassis-link"/>
+    <child link="front-right-wheel-link"/>
+    <origin rpy="0 0 0" xyz="0.042 0.065 0"/>
+    <axis xyz="0 1 0"/>
+  </joint>
+  <!-- ${x_position}-${y_position}-wheel-link -->
+  <link name="front-left-wheel-link">
+    <visual>
+      <origin rpy="1.5707963267948966 0 0" xyz="0 0 0"/>
+      <geometry>
+        <cylinder length="0.01" radius="0.02"/>
+      </geometry>
+      <material name="blue"/>
+    </visual>
+    <collision>
+      <origin rpy="1.5707963267948966 0 0" xyz="0 0 0"/>
+      <geometry>
+        <cylinder length="0.01" radius="0.02"/>
+      </geometry>
+    </collision>
+    <inertial>
+      <origin rpy="1.5707963267948966 0 0" xyz="0 0 0"/>
+      <mass value="0.2"/>
+      <inertia ixx="2.166666666666667e-05" ixy="0" ixz="0" iyy="2.166666666666667e-05" iyz="0" izz="4e-05"/>
+    </inertial>
+  </link>
+  <joint name="joint-chassis-front-left-wheel" type="continuous">
+    <parent link="chassis-link"/>
+    <child link="front-left-wheel-link"/>
+    <origin rpy="0 0 0" xyz="0.042 -0.065 0"/>
+    <axis xyz="0 1 0"/>
+  </joint>
+  <!-- ${x_position}-${y_position}-wheel-link -->
+  <link name="rare-right-wheel-link">
+    <visual>
+      <origin rpy="1.5707963267948966 0 0" xyz="0 0 0"/>
+      <geometry>
+        <cylinder length="0.01" radius="0.02"/>
+      </geometry>
+      <material name="blue"/>
+    </visual>
+    <collision>
+      <origin rpy="1.5707963267948966 0 0" xyz="0 0 0"/>
+      <geometry>
+        <cylinder length="0.01" radius="0.02"/>
+      </geometry>
+    </collision>
+    <inertial>
+      <origin rpy="1.5707963267948966 0 0" xyz="0 0 0"/>
+      <mass value="0.2"/>
+      <inertia ixx="2.166666666666667e-05" ixy="0" ixz="0" iyy="2.166666666666667e-05" iyz="0" izz="4e-05"/>
+    </inertial>
+  </link>
+  <joint name="joint-chassis-rare-right-wheel" type="continuous">
+    <parent link="chassis-link"/>
+    <child link="rare-right-wheel-link"/>
+    <origin rpy="0 0 0" xyz="-0.042 0.065 0"/>
+    <axis xyz="0 1 0"/>
+  </joint>
+  <!-- ${x_position}-${y_position}-wheel-link -->
+  <link name="rare-left-wheel-link">
+    <visual>
+      <origin rpy="1.5707963267948966 0 0" xyz="0 0 0"/>
+      <geometry>
+        <cylinder length="0.01" radius="0.02"/>
+      </geometry>
+      <material name="blue"/>
+    </visual>
+    <collision>
+      <origin rpy="1.5707963267948966 0 0" xyz="0 0 0"/>
+      <geometry>
+        <cylinder length="0.01" radius="0.02"/>
+      </geometry>
+    </collision>
+    <inertial>
+      <origin rpy="1.5707963267948966 0 0" xyz="0 0 0"/>
+      <mass value="0.2"/>
+      <inertia ixx="2.166666666666667e-05" ixy="0" ixz="0" iyy="2.166666666666667e-05" iyz="0" izz="4e-05"/>
+    </inertial>
+  </link>
+  <joint name="joint-chassis-rare-left-wheel" type="continuous">
+    <parent link="chassis-link"/>
+    <child link="rare-left-wheel-link"/>
+    <origin rpy="0 0 0" xyz="-0.042 -0.065 0"/>
+    <axis xyz="0 1 0"/>
+  </joint>
+  <gazebo reference="chassis-link">
+    <material>Gazebo/DarkGrey</material>
+  </gazebo>
+  <gazebo>
+  <gazebo reference="front-right-wheel-link">
+    <mu1>10000.0 </mu1>
+    <mu2>10000.0 </mu2>
+    <material>Gazebo/Purple</material>
+  </gazebo>
+  <gazebo reference="front-left-wheel-link">
+    <mu1>10000.0 </mu1>
+    <mu2>10000.0 </mu2>
+    <material>Gazebo/Purple</material>
+  </gazebo>
+  <gazebo reference="rare-right-wheel-link">
+    <mu1>10000.0 </mu1>
+    <mu2>10000.0 </mu2>
+    <material>Gazebo/Purple</material>
+  </gazebo>
+  <gazebo reference="rare-left-wheel-link">
+    <mu1>10000.0 </mu1>
+    <mu2>10000.0 </mu2>
+    <material>Gazebo/Purple</material>
+  </gazebo>
 </robot>

File: description/ros2_control.xacro (robot description, xacro)
@@ -5,5 +5,5 @@
                 <plugin>gz_ros2_control/GazeboSimSystem</plugin>
             </hardware>
-            <joint name="left_wheel_joint">
+            <joint name="joint-chassis-front-left-wheel">
                 <command_interface name="velocity">
                     <param name="min">-10</param>
@@ -13,5 +13,21 @@
                 <state_interface name="position"/>
             </joint>
-            <joint name="right_wheel_joint">
+            <joint name="joint-chassis-front-right-wheel">
+                <command_interface name="velocity">
+                    <param name="min">-10</param>
+                    <param name="max">10</param>
+                </command_interface>
+                <state_interface name="velocity"/>
+                <state_interface name="position"/>
+            </joint>
+            <joint name="joint-chassis-rare-right-wheel">
+                <command_interface name="velocity">
+                    <param name="min">-10</param>
+                    <param name="max">10</param>
+                </command_interface>
+                <state_interface name="velocity"/>
+                <state_interface name="position"/>
+            </joint>
+            <joint name="joint-chassis-rare-left-wheel">
                 <command_interface name="velocity">
                     <param name="min">-10</param>
