Commit message: 

File: description/robot.urdf.xacro (robot description, xacro)
@@ -2,3 +2,4 @@
 <robot xmlns:xacro="http://www.ros.org/wiki/xacro"  name="robot">
     <xacro:include filename="robot_core.xacro" />
+    <xacro:include filename="gazebo_control.xacro" />
 </robot>

File: description/robot_core.xacro (robot description, xacro)
@@ -41,4 +41,7 @@
         </xacro:inertial_box>
     </link>
+    <gazebo reference="chassis">
+        <material>Gazebo/White</material>
+    </gazebo>
     <!-- LEFT WHEEL LINK -->
     <joint name="left_wheel_joint" type="continuous">
@@ -64,4 +67,7 @@
         </xacro:inertial_cylinder>
     </link>
+    <gazebo reference="left_wheel">
+        <material>Gazebo/Blue</material>
+    </gazebo>
     <!-- RIGHT WHEEL LINK -->
     <joint name="right_wheel_joint" type="continuous">
@@ -87,4 +93,7 @@
         </xacro:inertial_cylinder>
     </link>
+    <gazebo reference="right_wheel">
+        <material>Gazebo/Blue</material>
+    </gazebo>
     <!-- CASTER WHEEL LINK -->
     <joint name="caster_wheel_joint" type="fixed">
@@ -109,3 +118,8 @@
         </xacro:inertial_sphere>
     </link>
+    <gazebo reference="caster_wheel">
+        <material>Gazebo/Black</material>
+        <mu1 value="0.001"/>
+        <mu2 value="0.001"/>
+    </gazebo>
 </robot>

Commit message: 

File: description/robot.urdf.xacro (robot description, xacro)
@@ -2,4 +2,3 @@
 <robot xmlns:xacro="http://www.ros.org/wiki/xacro"  name="robot">
     <xacro:include filename="robot_core.xacro" />
-    <xacro:include filename="gazebo_control.xacro" />
 </robot>

File: description/robot_core.xacro (robot description, xacro)
@@ -2,4 +2,6 @@
 <robot xmlns:xacro="http://www.ros.org/wiki/xacro" >
     <xacro:include filename="inertial_macros.xacro"/>
+    <!-- Add ros2_control xacro include -->
+    <xacro:include filename="$(find ros2_control_xacro_utils)/xacro/ros2_control.xacro" />
     <material name="white">
         <color rgba="1 1 1 1" />
@@ -123,3 +125,32 @@
         <mu2 value="0.001"/>
     </gazebo>
+    <!-- ========== ROS2 CONTROL CONFIGURATION ========== -->
+    <ros2_control name="diff_drive_robot" type="system">
+        <hardware>
+            <plugin>gz_ros2_control/GazeboSystem</plugin>
+        </hardware>
+        <joint name="left_wheel_joint">
+            <command_interface name="velocity">
+                <param name="min">-10.0</param>
+                <param name="max">10.0</param>
+            </command_interface>
+            <state_interface name="position"/>
+            <state_interface name="velocity"/>
+        </joint>
+        <joint name="right_wheel_joint">
+            <command_interface name="velocity">
+                <param name="min">-10.0</param>
+                <param name="max">10.0</param>
+            </command_interface>
+            <state_interface name="position"/>
+            <state_interface name="velocity"/>
+        </joint>
+    </ros2_control>
+    <!-- ========== GAZEBO ROS2 CONTROL PLUGIN ========== -->
+    <gazebo>
+        <plugin filename="libgz_ros2_control-system.so" name="gz_ros2_control::GazeboSystem">
+            <parameters>$(find my_bot)/config/diff_drive_controllers.yaml</parameters>
+            <controller_manager>controller_manager</controller_manager>
+        </plugin>
+    </gazebo>
 </robot>

Commit message: 

File: description/robot.urdf.xacro (robot description, xacro)
@@ -4,9 +4,4 @@
     <xacro:arg name="sim_mode" default="false"/>
     <xacro:include filename="robot_core.xacro" />
-    <xacro:if value="$(arg use_ros2_control)">
-        <xacro:include filename="ros2_control.xacro" />
-    </xacro:if>
-    <xacro:unless value="$(arg use_ros2_control)">
-        <xacro:include filename="gazebo_control.xacro" />
-    </xacro:unless>
+    <xacro:include filename="ros2_control.xacro" />
 </robot>

File: description/ros2_control.xacro (robot description, xacro)
@@ -1,34 +1,4 @@
 <?xml version="1.0"?>
 <robot xmlns:xacro="http://www.ros.org/wiki/xacro">
-    <xacro:unless value="$(arg sim_mode)">
-        <ros2_control name="RealRobot" type="system">
-            <hardware>
-                <plugin>diffdrive_arduino/DiffDriveArduinoHardware</plugin>
-                <param name="left_wheel_name">left_wheel_joint</param>
-                <param name="right_wheel_name">right_wheel_joint</param>
-                <param name="loop_rate">30</param>
-                <param name="device">/dev/ttyUSB0</param>
-                <param name="baud_rate">57600</param>
-                <param name="timeout_ms">1000</param>
-                <param name="enc_counts_per_rev">3436</param>
-            </hardware>
-            <joint name="left_wheel_joint">
-                <command_interface name="velocity">
-                    <param name="min">-10</param>
-                    <param name="max">10</param>
-                </command_interface>
-                <state_interface name="position"/>
-                <state_interface name="velocity"/>
-            </joint>
-            <joint name="right_wheel_joint">
-                <command_interface name="velocity">
-                    <param name="min">-10</param>
-                    <param name="max">10</param>
-                </command_interface>
-                <state_interface name="position"/>
-                <state_interface name="velocity"/>
-            </joint>
-        </ros2_control>
-    </xacro:unless>
     <xacro:if value="$(arg sim_mode)">
         <ros2_control name="GazeboSystem" type="system">

Commit message: 

File: description/robot.urdf.xacro (robot description, xacro)
@@ -5,3 +5,4 @@
     <xacro:include filename="robot_core.xacro" />
     <xacro:include filename="ros2_control.xacro" />
+    <xacro:include filename="lidar.xacro" />
 </robot>

File: description/robot_core.xacro (robot description, xacro)
@@ -1,4 +1,19 @@
 <?xml version="1.0"?>
 <robot xmlns:xacro="http://www.ros.org/wiki/xacro" >
+   <material name="white">
+        <color rgba="1 1 1 1" />
+   </material>
+    <material name="orange">
+        <color rgba="1 0.3 0.1 1"/>
+    </material>
+    <material name="blue">
+        <color rgba="0.2 0.2 1 1"/>
+    </material>
+    <material name="black">
+        <color rgba="0 0 0 1"/>
+    </material>
+    <material name="red">
+        <color rgba="1 0 0 1"/>
+    </material>
   <!--dummy link-->
   <link name="base_link"/>

Commit message: 

File: description/robot.urdf.xacro (robot description, xacro)
@@ -5,4 +5,3 @@
     <xacro:include filename="robot_core.xacro" />
     <xacro:include filename="ros2_control.xacro" />
-    <xacro:include filename="lidar.xacro" />
 </robot>

File: description/robot_core.xacro (robot description, xacro)
@@ -1,5 +1,5 @@
 <?xml version="1.0"?>
 <robot xmlns:xacro="http://www.ros.org/wiki/xacro" >
-<!-- BASE LINK -->
+  <!-- BASE LINK -->
   <link name="base_link">
   </link>
@@ -17,5 +17,6 @@
       <origin rpy="0 0 0" xyz="0 0 0"/>
       <geometry>
-        <box size="0.14 0.12 0.01"/>
+        <!-- from PDF: ~120.02 x 112.87 x 10 mm -->
+        <box size="0.12002 0.11287 0.01"/>
       </geometry>
       <material name="brown">
@@ -26,10 +27,11 @@
       <origin rpy="0 0 0" xyz="0 0 0"/>
       <geometry>
-        <box size="0.14 0.12 0.01"/>
+        <box size="0.12002 0.11287 0.01"/>
       </geometry>
     </collision>
     <inertial>
-      <mass value="0.4"/>
-      <inertia ixx="0.00048333" ixy="0" ixz="0" iyy="0.0013367" iyz="0" izz="0.0018133"/>
+      <mass value="0.6"/>
+      <!-- box inertia about its center: ixx=m*(y^2+z^2)/12 etc. -->
+      <inertia ixx="0.000641981845" ixy="0" ixz="0" iyy="0.00072524002" iyz="0" izz="0.001357221865"/>
     </inertial>
   </link>
@@ -37,4 +39,5 @@
     <parent link="base_link"/>
     <child link="chassis-link"/>
+    <!-- keep same height reference as your original (raise chassis center 20 mm) -->
     <origin rpy="0 0 0" xyz="0 0 0.02"/>
   </joint>
@@ -47,5 +50,6 @@
       <origin rpy="1.5707963267948966 0 0" xyz="0 0 0"/>
       <geometry>
-        <cylinder length="0.01" radius="0.02"/>
+        <!-- from PDF: wheel Ø~58 mm, width ~12 mm -->
+        <cylinder length="0.012" radius="0.029"/>
       </geometry>
       <material name="blue"/>
@@ -54,11 +58,11 @@
       <origin rpy="1.5707963267948966 0 0" xyz="0 0 0"/>
       <geometry>
-        <cylinder length="0.01" radius="0.02"/>
+        <cylinder length="0.012" radius="0.029"/>
       </geometry>
     </collision>
     <inertial>
       <origin rpy="1.5707963267948966 0 0" xyz="0 0 0"/>
-      <mass value="0.2"/>
-      <inertia ixx="2.166666666666667e-05" ixy="0" ixz="0" iyy="2.166666666666667e-05" iyz="0" izz="4e-05"/>
+      <mass value="0.15"/>
+      <inertia ixx="3.33375e-05" ixy="0" ixz="0" iyy="3.33375e-05" iyz="0" izz="6.3075e-05"/>
     </inertial>
   </link>
@@ -66,5 +70,6 @@
     <parent link="chassis-link"/>
     <child link="front-right-wheel-link"/>
-    <origin rpy="0 0 0" xyz="0.042 0.065 0"/>
+    <!-- place wheel centers near the corners using new chassis size -->
+    <origin rpy="0 0 0" xyz="0.03101 0.051435 0"/>
     <axis xyz="0 1 0"/>
   </joint>
@@ -74,5 +79,5 @@
       <origin rpy="1.5707963267948966 0 0" xyz="0 0 0"/>
       <geometry>
-        <cylinder length="0.01" radius="0.02"/>
+        <cylinder length="0.012" radius="0.029"/>
       </geometry>
       <material name="blue"/>
@@ -81,11 +86,11 @@
       <origin rpy="1.5707963267948966 0 0" xyz="0 0 0"/>
       <geometry>
-        <cylinder length="0.01" radius="0.02"/>
+        <cylinder length="0.012" radius="0.029"/>
       </geometry>
     </collision>
     <inertial>
       <origin rpy="1.5707963267948966 0 0" xyz="0 0 0"/>
-      <mass value="0.2"/>
-      <inertia ixx="2.166666666666667e-05" ixy="0" ixz="0" iyy="2.166666666666667e-05" iyz="0" izz="4e-05"/>
+      <mass value="0.15"/>
+      <inertia ixx="3.33375e-05" ixy="0" ixz="0" iyy="3.33375e-05" iyz="0" izz="6.3075e-05"/>
     </inertial>
   </link>
@@ -93,5 +98,5 @@
     <parent link="chassis-link"/>
     <child link="front-left-wheel-link"/>
-    <origin rpy="0 0 0" xyz="0.042 -0.065 0"/>
+    <origin rpy="0 0 0" xyz="0.03101 -0.051435 0"/>
     <axis xyz="0 1 0"/>
   </joint>
@@ -101,5 +106,5 @@
       <origin rpy="1.5707963267948966 0 0" xyz="0 0 0"/>
       <geometry>
-        <cylinder length="0.01" radius="0.02"/>
+        <cylinder length="0.012" radius="0.029"/>
       </geometry>
       <material name="blue"/>
@@ -108,11 +113,11 @@
       <origin rpy="1.5707963267948966 0 0" xyz="0 0 0"/>
       <geometry>
-        <cylinder length="0.01" radius="0.02"/>
+        <cylinder length="0.012" radius="0.029"/>
       </geometry>
     </collision>
     <inertial>
       <origin rpy="1.5707963267948966 0 0" xyz="0 0 0"/>
-      <mass value="0.2"/>
-      <inertia ixx="2.166666666666667e-05" ixy="0" ixz="0" iyy="2.166666666666667e-05" iyz="0" izz="4e-05"/>
+      <mass value="0.15"/>
+      <inertia ixx="3.33375e-05" ixy="0" ixz="0" iyy="3.33375e-05" iyz="0" izz="6.3075e-05"/>
     </inertial>
   </link>
@@ -120,5 +125,5 @@
     <parent link="chassis-link"/>
     <child link="rare-right-wheel-link"/>
-    <origin rpy="0 0 0" xyz="-0.042 0.065 0"/>
+    <origin rpy="0 0 0" xyz="-0.03101 0.051435 0"/>
     <axis xyz="0 1 0"/>
   </joint>
@@ -128,5 +133,5 @@
       <origin rpy="1.5707963267948966 0 0" xyz="0 0 0"/>
       <geometry>
-        <cylinder length="0.01" radius="0.02"/>
+        <cylinder length="0.012" radius="0.029"/>
       </geometry>
       <material name="blue"/>
@@ -135,11 +140,11 @@
       <origin rpy="1.5707963267948966 0 0" xyz="0 0 0"/>
       <geometry>
-        <cylinder length="0.01" radius="0.02"/>
+        <cylinder length="0.012" radius="0.029"/>
       </geometry>
     </collision>
     <inertial>
       <origin rpy="1.5707963267948966 0 0" xyz="0 0 0"/>
-      <mass value="0.2"/>
-      <inertia ixx="2.166666666666667e-05" ixy="0" ixz="0" iyy="2.166666666666667e-05" iyz="0" izz="4e-05"/>
+      <mass value="0.15"/>
+      <inertia ixx="3.33375e-05" ixy="0" ixz="0" iyy="3.33375e-05" iyz="0" izz="6.3075e-05"/>
     </inertial>
   </link>
@@ -147,5 +152,5 @@
     <parent link="chassis-link"/>
     <child link="rare-left-wheel-link"/>
-    <origin rpy="0 0 0" xyz="-0.042 -0.065 0"/>
+    <origin rpy="0 0 0" xyz="-0.03101 -0.051435 0"/>
     <axis xyz="0 1 0"/>
   </joint>
