Commit message: 

File: description/lidar.xacro (robot description, xacro)
@@ -13,5 +13,5 @@
             <cylinder radius="0.05" length="0.04"/>
         </geometry>
-        <material name="black"/>
+        <material name="blue"/>
     </visual>
     <visual>
@@ -20,5 +20,5 @@
             <cylinder radius="0.01" length="0.1"/>
         </geometry>
-        <material name="black"/>
+        <material name="blue"/>
     </visual>
     <collision>

File: description/robot.urdf.xacro (robot description, xacro)
@@ -5,4 +5,4 @@
     <xacro:include filename="robot_core.xacro" />
     <xacro:include filename="ros2_control.xacro" />
-   <!--  <xacro:include filename="lidar.xacro" />-->
+    <xacro:include filename="lidar.xacro" />
 </robot>

Commit message: 

File: description/lidar.xacro (robot description, xacro)
@@ -7,26 +7,14 @@
     <child link="laser_frame"/>
     <!-- place laser centered on chassis and slightly above -->
-    <origin xyz="0 0 0.02" rpy="0 0 0"/>
+    <origin xyz="0 0 0.04" rpy="0 0 0"/>
 </joint>
 <link name="laser_frame">
     <visual>
         <geometry>
-            <cylinder radius="0.05" length="0.04"/>
+            <cylinder radius="0.03" length="0.03"/>
         </geometry>
         <material name="blue"/>
     </visual>
-    <visual>
-        <origin xyz="0 0 -0.05"/>
-        <geometry>
-            <cylinder radius="0.01" length="0.1"/>
-        </geometry>
-        <material name="blue"/>
-    </visual>
-    <collision>
-        <geometry>
-            <cylinder radius="0.05" length="0.04"/>
-        </geometry>
-    </collision>
-    <xacro:inertial_cylinder mass="0.1" length="0.04" radius="0.05">
+    <xacro:inertial_cylinder mass="0.01" length="0.0003" radius="0.002">
         <origin xyz="0 0 0" rpy="0 0 0"/>
     </xacro:inertial_cylinder>

Commit message: 

File: description/lidar.xacro (robot description, xacro)
@@ -7,10 +7,10 @@
     <child link="laser_frame"/>
     <!-- place laser centered on chassis and slightly above -->
-    <origin xyz="0 0 0.04" rpy="0 0 0"/>
+    <origin xyz="0 0 0.02" rpy="0 0 0"/>
 </joint>
 <link name="laser_frame">
     <visual>
         <geometry>
-            <cylinder radius="0.03" length="0.03"/>
+            <cylinder radius="0.01" length="0.001"/>
         </geometry>
         <material name="blue"/>

Commit message: 

File: description/lidar.xacro (robot description, xacro)
@@ -7,10 +7,10 @@
     <child link="laser_frame"/>
     <!-- place laser centered on chassis and slightly above -->
-    <origin xyz="0 0 0.02" rpy="0 0 0"/>
+    <origin xyz="0 0 0" rpy="0 0 0"/>
 </joint>
 <link name="laser_frame">
     <visual>
         <geometry>
-            <cylinder radius="0.01" length="0.001"/>
+            <cylinder radius="0.01" length="0.03"/>
         </geometry>
         <material name="blue"/>

Commit message: 

File: description/lidar.xacro (robot description, xacro)
@@ -7,5 +7,5 @@
     <child link="laser_frame"/>
     <!-- place laser centered on chassis and slightly above -->
-    <origin xyz="0 0 0" rpy="0 0 0"/>
+    <origin xyz="0 0 0.01" rpy="0 0 0"/>
 </joint>
 <link name="laser_frame">

Commit message: 

File: description/lidar.xacro (robot description, xacro)
@@ -7,5 +7,5 @@
     <child link="laser_frame"/>
     <!-- place laser centered on chassis and slightly above -->
-    <origin xyz="0 0 0.01" rpy="0 0 0"/>
+    <origin xyz="0 0 0.02" rpy="0 0 0"/>
 </joint>
 <link name="laser_frame">
@@ -16,4 +16,16 @@
         <material name="blue"/>
     </visual>
+    <visual>
+        <origin xyz="0 0 -0.005"/>
+        <geometry>
+            <cylinder radius="0.01" length="0.1"/>
+        </geometry>
+        <material name="blue"/>
+    </visual>
+    <collision>
+        <geometry>
+            <cylinder radius="0.05" length="0.04"/>
+        </geometry>
+    </collision>
     <xacro:inertial_cylinder mass="0.01" length="0.0003" radius="0.002">
         <origin xyz="0 0 0" rpy="0 0 0"/>

Commit message: 

File: description/lidar.xacro (robot description, xacro)
@@ -1,70 +1,54 @@
-<?xml version="1.0"?>
-<robot xmlns:xacro="http://www.ros.org/wiki/xacro" >
-<xacro:include filename="inertial_macros.xacro"/>
-<!-- Laser mounted on top of chassis -->
-<joint name="laser_joint" type="fixed">
-    <parent link="chassis-link"/>
-    <child link="laser_frame"/>
-    <!-- place laser centered on chassis and slightly above -->
-    <origin xyz="0 0 0.02" rpy="0 0 0"/>
-</joint>
-<link name="laser_frame">
+  <!-- LiDAR link centered above the chassis -->
+  <link name="lidar_link">
     <visual>
-        <geometry>
-            <cylinder radius="0.01" length="0.03"/>
-        </geometry>
-        <material name="blue"/>
-    </visual>
-    <visual>
-        <origin xyz="0 0 -0.005"/>
-        <geometry>
-            <cylinder radius="0.01" length="0.1"/>
-        </geometry>
-        <material name="blue"/>
+      <origin xyz="0 0 0" rpy="0 0 0"/>
+      <geometry><cylinder radius="0.025" length="0.02"/></geometry>
+      <material name="blue"/>
     </visual>
     <collision>
-        <geometry>
-            <cylinder radius="0.05" length="0.04"/>
-        </geometry>
+      <origin xyz="0 0 0" rpy="0 0 0"/>
+      <geometry><cylinder radius="0.025" length="0.02"/></geometry>
     </collision>
-    <xacro:inertial_cylinder mass="0.01" length="0.0003" radius="0.002">
-        <origin xyz="0 0 0" rpy="0 0 0"/>
-    </xacro:inertial_cylinder>
-</link>
-<gazebo reference="laser_frame">
-    <material>Gazebo/Black</material>
-    <plugin
-      filename="libignition-gazebo-sensors-system.so"
-      name="ignition::gazebo::systems::Sensors">
-      <render_engine>ogre2</render_engine>
-    </plugin>
-    <sensor name='gpu_lidar' type='gpu_lidar'>"
-    <pose relative_to='lidar_frame'>0 0 0 0 0 0</pose>
-    <topic>lidar</topic>
-    <update_rate>10</update_rate>
-    <ray>
+    <inertial>
+      <origin xyz="0 0 0" rpy="0 0 0"/>
+      <mass value="0.15"/>
+      <inertia ixx="1e-4" ixy="0" ixz="0" iyy="1e-4" iyz="0" izz="1e-4"/>
+    </inertial>
+  </link>
+  <!-- Fixed mount: centered in X/Y, 6 cm above the chassis top -->
+  <joint name="joint-chassis-lidar" type="fixed">
+    <parent link="chassis-link"/>
+    <child link="lidar_link"/>
+    <origin xyz="0 0 0.06" rpy="0 0 0"/>
+  </joint>
+  <!-- Gazebo Fortress (gz-sim) sensor: GPU lidar publishing on a gz transport topic -->
+  <gazebo reference="lidar_link">
+    <sensor name="lidar" type="gpu_lidar">
+      <update_rate>20</update_rate>
+      <!-- Pose of the scan frame within lidar_link -->
+      <pose>0 0 0 0 0 0</pose>
+      <ray>
         <scan>
-            <horizontal>
-                <samples>640</samples>
-                <resolution>1</resolution>
-                <min_angle>-1.396263</min_angle>
-                <max_angle>1.396263</max_angle>
-            </horizontal>
-            <vertical>
-                <samples>1</samples>
-                <resolution>0.01</resolution>
-                <min_angle>0</min_angle>
-                <max_angle>0</max_angle>
-            </vertical>
+          <horizontal>
+            <!-- 360° FoV with ~0.5° resolution -->
+            <samples>720</samples>
+            <resolution>1</resolution>
+            <min_angle>-3.14159265359</min_angle>
+            <max_angle> 3.14159265359</max_angle>
+          </horizontal>
         </scan>
         <range>
-            <min>0.08</min>
-            <max>10.0</max>
-            <resolution>0.01</resolution>
+          <min>0.12</min>
+          <max>12.0</max>
+          <resolution>0.01</resolution>
         </range>
-    </ray>
-    <always_on>1</always_on>
-    <visualize>true</visualize>
+        <noise>
+          <type>gaussian</type>
+          <mean>0.0</mean>
+          <stddev>0.01</stddev>
+        </noise>
+      </ray>
+      <!-- Optional: set a custom gz transport topic (otherwise an auto one is used) -->
+      <topic>/lidar/scan</topic>
     </sensor>
-</gazebo>
-</robot>
+  </gazebo>

Commit message: 

File: description/lidar.xacro (robot description, xacro)
@@ -22,5 +22,5 @@
     <parent link="chassis-link"/>
     <child link="lidar_link"/>
-    <origin xyz="0 0 0.06" rpy="0 0 0"/>
+    <origin xyz="0 0 0.03" rpy="0 0 0"/>
   </joint>
   <!-- Gazebo Fortress (gz-sim) sensor: GPU lidar publishing on a gz transport topic -->
@@ -52,5 +52,5 @@
       </ray>
       <!-- Optional: set a custom gz transport topic (otherwise an auto one is used) -->
-      <topic>/lidar/scan</topic>
+      <topic>/scan</topic>
     </sensor>
   </gazebo>

Commit message: 

File: description/lidar.xacro (robot description, xacro)
@@ -22,5 +22,5 @@
     <parent link="chassis-link"/>
     <child link="lidar_link"/>
-    <origin xyz="0 0 0.03" rpy="0 0 0"/>
+    <origin xyz="0 0 0.005" rpy="0 0 0"/>
   </joint>
   <!-- Gazebo Fortress (gz-sim) sensor: GPU lidar publishing on a gz transport topic -->
@@ -54,4 +54,5 @@
       <!-- Optional: set a custom gz transport topic (otherwise an auto one is used) -->
       <topic>/scan</topic>
+      <frame_id>lidar_link</frame_id>
     </sensor>
   </gazebo>

Commit message: 

File: description/lidar.xacro (robot description, xacro)
@@ -2,5 +2,5 @@
 <robot xmlns:xacro="http://www.ros.org/wiki/xacro" >
   <!-- LiDAR link centered above the chassis -->
-  <link name="lidar_link">
+  <link name="laser_frame">
     <visual>
       <origin xyz="0 0 0" rpy="0 0 0"/>
@@ -21,44 +21,30 @@
   <joint name="joint-chassis-lidar" type="fixed">
     <parent link="chassis-link"/>
-    <child link="lidar_link"/>
+    <child link="laser_frame"/>
     <origin xyz="0 0 0.005" rpy="0 0 0"/>
   </joint>
   <!-- Gazebo Fortress (gz-sim) sensor: GPU lidar publishing on a gz transport topic -->
-  <gazebo reference="lidar_link">
-    <sensor name='gpu_lidar' type='gpu_lidar'>"
-    <pose relative_to='lidar_frame'>0 0 0 0 0 0</pose>
-    <topic>/scan</topic>
-    <update_rate>10</update_rate>
-    <ray>
-        <scan>
-            <horizontal>
-                <samples>640</samples>
-                <resolution>1</resolution>
-                <min_angle>-1.396263</min_angle>
-                <max_angle>1.396263</max_angle>
-            </horizontal>
-            <vertical>
-                <samples>1</samples>
-                <resolution>0.01</resolution>
-                <min_angle>0</min_angle>
-                <max_angle>0</max_angle>
-            </vertical>
-        </scan>
-        <range>
-            <min>0.08</min>
-            <max>10.0</max>
-            <resolution>0.01</resolution>
-        </range>
-      </ray>
-      <always_on>1</always_on>
-      <visualize>true</visualize>
-      <plugin name="laser_controller" filename="libgazebo_ros_ray_sensor.so">
-                <ros>
-                    <argument>~/out:=/scan</argument>
-                </ros>
-                <output_type>sensor_msgs/LaserScan</output_type>
-                <frame_name>laser_frame</frame_name>
-      </plugin>
-     </sensor>
-  </gazebo>
+ <gazebo reference="laser_frame">
+        <material>Gazebo/Black</material>
+        <sensor name="laser" type="gpu_lidar">
+            <pose> 0 0 0 0 0 0 </pose>
+            <visualize>false</visualize>
+            <update_rate>10</update_rate>
+            <lidar>
+                <scan>
+                    <horizontal>
+                        <samples>360</samples>
+                        <min_angle>-3.14</min_angle>
+                        <max_angle>3.14</max_angle>
+                    </horizontal>
+                </scan>
+                <range>
+                    <min>0.3</min>
+                    <max>12</max>
+                </range>
+            </lidar>
+            <topic>scan</topic>
+            <gz_frame_id>laser_frame</gz_frame_id>
+        </sensor>
+    </gazebo>
 </robot>

Commit message: 

File: description/lidar.xacro (robot description, xacro)
@@ -22,5 +22,5 @@
     <parent link="chassis-link"/>
     <child link="laser_frame"/>
-    <origin xyz="0 0 0.005" rpy="0 0 0"/>
+    <origin xyz="0 0 0.01" rpy="0 0 0"/>
   </joint>
   <!-- Gazebo Fortress (gz-sim) sensor: GPU lidar publishing on a gz transport topic -->

Commit message: 

File: description/lidar.xacro (robot description, xacro)
@@ -10,5 +10,5 @@
     <collision>
       <origin xyz="0 0 0" rpy="0 0 0"/>
-      <geometry><cylinder radius="0.025" length="0.02"/></geometry>
+      <geometry><cylinder radius="0.025" length="0.04"/></geometry>
     </collision>
     <inertial>
@@ -22,5 +22,5 @@
     <parent link="chassis-link"/>
     <child link="laser_frame"/>
-    <origin xyz="0 0 0.01" rpy="0 0 0"/>
+    <origin xyz="0 0 0.03" rpy="0 0 0"/>
   </joint>
   <!-- Gazebo Fortress (gz-sim) sensor: GPU lidar publishing on a gz transport topic -->

Commit message: 

File: description/lidar.xacro (robot description, xacro)
@@ -1,26 +1,43 @@
 <?xml version="1.0"?>
 <robot xmlns:xacro="http://www.ros.org/wiki/xacro" >
-  <!-- LiDAR link centered above the chassis -->
-  <link name="laser_frame">
+  <!-- ========= LiDAR "inside chassis" with an optical frame above top ======== -->
+  <!-- 1) A hidden LiDAR body inside the chassis (visual only, tiny collision) -->
+  <link name="lidar_body">
     <visual>
-      <origin xyz="0 0 0" rpy="0 0 0"/>
-      <geometry><cylinder radius="0.025" length="0.02"/></geometry>
+      <!-- Put the can inside the 10 mm-thick chassis plate -->
+      <!-- chassis center is at z=0.02, thickness=0.01 -> top at 0.025 -->
+      <origin xyz="0 0 0.02" rpy="0 0 0"/>
+      <geometry>
+        <cylinder radius="0.025" length="0.02"/>
+      </geometry>
       <material name="blue"/>
     </visual>
     <collision>
-      <origin xyz="0 0 0" rpy="0 0 0"/>
-      <geometry><cylinder radius="0.025" length="0.04"/></geometry>
+      <!-- Tiny collision so it doesn't interfere with rays -->
+      <origin xyz="0 0 0.02" rpy="0 0 0"/>
+      <geometry>
+        <sphere radius="0.001"/>
+      </geometry>
     </collision>
     <inertial>
-      <origin xyz="0 0 0" rpy="0 0 0"/>
+      <origin xyz="0 0 0.02" rpy="0 0 0"/>
       <mass value="0.15"/>
       <inertia ixx="1e-4" ixy="0" ixz="0" iyy="1e-4" iyz="0" izz="1e-4"/>
     </inertial>
   </link>
-  <!-- Fixed mount: centered in X/Y, 6 cm above the chassis top -->
-  <joint name="joint-chassis-lidar" type="fixed">
+  <!-- Fixed mount: lidar_body is bolted to the chassis center -->
+  <joint name="joint-chassis-lidar_body" type="fixed">
     <parent link="chassis-link"/>
-    <child link="laser_frame"/>
-    <origin xyz="0 0 0.03" rpy="0 0 0"/>
+    <child  link="lidar_body"/>
+    <origin xyz="0 0 0" rpy="0 0 0"/>
+  </joint>
+  <!-- 2) The optical frame (where the scan originates) just above the chassis top -->
+  <link name="laser_frame"/>
+  <joint name="joint-lidar_body-laser_frame" type="fixed">
+    <parent link="lidar_body"/>
+    <!-- Place the optical frame slightly above the top surface to avoid self-hits -->
+    <!-- chassis top = 0.025; put optical frame at 0.028 (3 mm clearance) -->
+    <child  link="laser_frame"/>
+    <origin xyz="0 0 0.008" rpy="0 0 0"/>
   </joint>
   <!-- Gazebo Fortress (gz-sim) sensor: GPU lidar publishing on a gz transport topic -->

Commit message: 

File: description/lidar.xacro (robot description, xacro)
@@ -30,5 +30,5 @@
     <parent link="chassis-link"/>
     <child  link="lidar_body"/>
-    <origin xyz="0 0 0" rpy="0 0 0"/>
+    <origin xyz="0 0 -0.1" rpy="0 0 0"/>
   </joint>
   <!-- 2) The optical frame (where the scan originates) just above the chassis top -->
@@ -39,5 +39,5 @@
     <!-- chassis top = 0.025; put optical frame at 0.028 (3 mm clearance) -->
     <child  link="laser_frame"/>
-    <origin xyz="0 0 0.008" rpy="0 0 0"/>
+    <origin xyz="0 0 0.01" rpy="0 0 0"/>
   </joint>
   <!-- Gazebo Fortress (gz-sim) sensor: GPU lidar publishing on a gz transport topic -->

Commit message: 

File: description/lidar.xacro (robot description, xacro)
@@ -9,5 +9,5 @@
       <origin xyz="0 0 0.02" rpy="0 0 0"/>
       <geometry>
-        <cylinder radius="0.025" length="0.02"/>
+        <cylinder radius="0.025" length="0.03"/>
       </geometry>
       <material name="blue"/>
@@ -30,5 +30,5 @@
     <parent link="chassis-link"/>
     <child  link="lidar_body"/>
-    <origin xyz="0 0 -0.1" rpy="0 0 0"/>
+    <origin xyz="0 0 -0.2" rpy="0 0 0"/>
   </joint>
   <!-- 2) The optical frame (where the scan originates) just above the chassis top -->

Commit message: 

File: description/lidar.xacro (robot description, xacro)
@@ -30,5 +30,5 @@
     <parent link="chassis-link"/>
     <child  link="lidar_body"/>
-    <origin xyz="0 0 -0.2" rpy="0 0 0"/>
+    <origin xyz="0 0 -0.1" rpy="0 0 0"/>
   </joint>
   <!-- 2) The optical frame (where the scan originates) just above the chassis top -->

Commit message: 

File: description/lidar.xacro (robot description, xacro)
@@ -30,5 +30,5 @@
     <parent link="chassis-link"/>
     <child  link="lidar_body"/>
-    <origin xyz="0 0 -0.1" rpy="0 0 0"/>
+    <origin xyz="0 0 0.09" rpy="0 0 0"/>
   </joint>
   <!-- 2) The optical frame (where the scan originates) just above the chassis top -->

Commit message: 

File: description/lidar.xacro (robot description, xacro)
@@ -30,5 +30,5 @@
     <parent link="chassis-link"/>
     <child  link="lidar_body"/>
-    <origin xyz="0 0 0.09" rpy="0 0 0"/>
+    <origin xyz="0 0 0" rpy="0 0 0"/>
   </joint>
   <!-- 2) The optical frame (where the scan originates) just above the chassis top -->

Commit message: 

File: description/lidar.xacro (robot description, xacro)
@@ -39,5 +39,5 @@
     <!-- chassis top = 0.025; put optical frame at 0.028 (3 mm clearance) -->
     <child  link="laser_frame"/>
-    <origin xyz="0 0 0.01" rpy="0 0 0"/>
+    <origin xyz="0 0 0.04" rpy="0 0 0"/>
   </joint>
   <!-- Gazebo Fortress (gz-sim) sensor: GPU lidar publishing on a gz transport topic -->

Commit message: 

File: description/lidar.xacro (robot description, xacro)
@@ -30,5 +30,5 @@
     <parent link="chassis-link"/>
     <child  link="lidar_body"/>
-    <origin xyz="0 0 0" rpy="0 0 0"/>
+    <origin xyz="0 0 0.04" rpy="0 0 0"/>
   </joint>
   <!-- 2) The optical frame (where the scan originates) just above the chassis top -->

Commit message: 

File: description/lidar.xacro (robot description, xacro)
@@ -39,5 +39,5 @@
     <!-- chassis top = 0.025; put optical frame at 0.028 (3 mm clearance) -->
     <child  link="laser_frame"/>
-    <origin xyz="0 0 0.04" rpy="0 0 0"/>
+    <origin xyz="0 0 0.02" rpy="0 0 0"/>
   </joint>
   <!-- Gazebo Fortress (gz-sim) sensor: GPU lidar publishing on a gz transport topic -->

Commit message: 

File: description/lidar.xacro (robot description, xacro)
@@ -30,5 +30,5 @@
     <parent link="chassis-link"/>
     <child  link="lidar_body"/>
-    <origin xyz="0 0 0.04" rpy="0 0 0"/>
+    <origin xyz="0 0 0" rpy="0 0 0"/>
   </joint>
   <!-- 2) The optical frame (where the scan originates) just above the chassis top -->

Commit message: 

File: description/lidar.xacro (robot description, xacro)
@@ -39,5 +39,5 @@
     <!-- chassis top = 0.025; put optical frame at 0.028 (3 mm clearance) -->
     <child  link="laser_frame"/>
-    <origin xyz="0 0 0.02" rpy="0 0 0"/>
+    <origin xyz="0 0 0" rpy="0 0 0"/>
   </joint>
   <!-- Gazebo Fortress (gz-sim) sensor: GPU lidar publishing on a gz transport topic -->

Commit message: 

File: description/lidar.xacro (robot description, xacro)
@@ -39,5 +39,5 @@
     <!-- chassis top = 0.025; put optical frame at 0.028 (3 mm clearance) -->
     <child  link="laser_frame"/>
-    <origin xyz="0 0 0" rpy="0 0 0"/>
+    <origin xyz="0 0 0.01" rpy="0 0 0"/>
   </joint>
   <!-- Gazebo Fortress (gz-sim) sensor: GPU lidar publishing on a gz transport topic -->

Commit message: 

File: description/lidar.xacro (robot description, xacro)
@@ -39,5 +39,5 @@
     <!-- chassis top = 0.025; put optical frame at 0.028 (3 mm clearance) -->
     <child  link="laser_frame"/>
-    <origin xyz="0 0 0.01" rpy="0 0 0"/>
+    <origin xyz="0 0 -0.01" rpy="0 0 0"/>
   </joint>
   <!-- Gazebo Fortress (gz-sim) sensor: GPU lidar publishing on a gz transport topic -->

Commit message: 

File: description/lidar.xacro (robot description, xacro)
@@ -39,5 +39,5 @@
     <!-- chassis top = 0.025; put optical frame at 0.028 (3 mm clearance) -->
     <child  link="laser_frame"/>
-    <origin xyz="0 0 -0.01" rpy="0 0 0"/>
+    <origin xyz="0 0 -0.028" rpy="0 0 0"/>
   </joint>
   <!-- Gazebo Fortress (gz-sim) sensor: GPU lidar publishing on a gz transport topic -->

Commit message: 

File: description/lidar.xacro (robot description, xacro)
@@ -39,5 +39,5 @@
     <!-- chassis top = 0.025; put optical frame at 0.028 (3 mm clearance) -->
     <child  link="laser_frame"/>
-    <origin xyz="0 0 -0.028" rpy="0 0 0"/>
+    <origin xyz="0 0 -0.03" rpy="0 0 0"/>
   </joint>
   <!-- Gazebo Fortress (gz-sim) sensor: GPU lidar publishing on a gz transport topic -->

Commit message: 

File: description/lidar.xacro (robot description, xacro)
@@ -39,5 +39,5 @@
     <!-- chassis top = 0.025; put optical frame at 0.028 (3 mm clearance) -->
     <child  link="laser_frame"/>
-    <origin xyz="0 0 -0.03" rpy="0 0 0"/>
+    <origin xyz="0 0 -0.04" rpy="0 0 0"/>
   </joint>
   <!-- Gazebo Fortress (gz-sim) sensor: GPU lidar publishing on a gz transport topic -->
