Commit message: 

File: description/lidar.xacro (robot description, xacro)
@@ -1,46 +1,38 @@
 <?xml version="1.0"?>
 <robot xmlns:xacro="http://www.ros.org/wiki/xacro" >
-  <!-- ========= LiDAR "inside chassis" with an optical frame above top ======== -->
-  <!-- 1) A hidden LiDAR body inside the chassis (visual only, tiny collision) -->
-  <link name="lidar_body">
+    <!-- ========= LiDAR "inside chassis" with an optical frame above top ======== -->
+  <!-- ===== LiDAR mount (centered above the chassis) ===== -->
+  <!-- LiDAR puck body -->
+  <link name="laser_frame">
     <visual>
-      <!-- Put the can inside the 10 mm-thick chassis plate -->
-      <!-- chassis center is at z=0.02, thickness=0.01 -> top at 0.025 -->
-      <origin xyz="0 0 0.02" rpy="0 0 0"/>
-      <geometry>
-        <cylinder radius="0.025" length="0.03"/>
-      </geometry>
-      <material name="blue"/>
+      <origin xyz="0 0 0" rpy="0 0 0"/>
+      <geometry><cylinder radius="0.05" length="0.04"/></geometry>
+      <material name="black"/>
+    </visual>
+    <!-- little mast (optional visual) -->
+    <visual>
+      <origin xyz="0 0 -0.05" rpy="0 0 0"/>
+      <geometry><cylinder radius="0.01" length="0.10"/></geometry>
+      <material name="black"/>
     </visual>
     <collision>
-      <!-- Tiny collision so it doesn't interfere with rays -->
-      <origin xyz="0 0 0.02" rpy="0 0 0"/>
-      <geometry>
-        <sphere radius="0.001"/>
-      </geometry>
+      <origin xyz="0 0 0" rpy="0 0 0"/>
+      <geometry><cylinder radius="0.05" length="0.04"/></geometry>
     </collision>
+    <!-- simple inertial; adjust if needed -->
     <inertial>
-      <origin xyz="0 0 0.02" rpy="0 0 0"/>
-      <mass value="0.15"/>
-      <inertia ixx="1e-4" ixy="0" ixz="0" iyy="1e-4" iyz="0" izz="1e-4"/>
+      <origin xyz="0 0 0" rpy="0 0 0"/>
+      <mass value="0.10"/>
+      <inertia ixx="1.0e-4" ixy="0" ixz="0" iyy="1.0e-4" iyz="0" izz="2.0e-4"/>
     </inertial>
   </link>
-  <!-- Fixed mount: lidar_body is bolted to the chassis center -->
-  <joint name="joint-chassis-lidar_body" type="fixed">
+  <!-- Fixed mount: centered in XY, raised in Z (6 cm above chassis top) -->
+  <joint name="joint-chassis-lidar" type="fixed">
     <parent link="chassis-link"/>
-    <child  link="lidar_body"/>
-    <origin xyz="0 0 0" rpy="0 0 0"/>
-  </joint>
-  <!-- 2) The optical frame (where the scan originates) just above the chassis top -->
-  <link name="laser_frame"/>
-  <joint name="joint-lidar_body-laser_frame" type="fixed">
-    <parent link="lidar_body"/>
-    <!-- Place the optical frame slightly above the top surface to avoid self-hits -->
-    <!-- chassis top = 0.025; put optical frame at 0.028 (3 mm clearance) -->
-    <child  link="laser_frame"/>
-    <origin xyz="0 0 -0.04" rpy="0 0 0"/>
+    <child link="laser_frame"/>
+    <origin xyz="0 0 0.06" rpy="0 0 0"/>
   </joint>
   <!-- Gazebo Fortress (gz-sim) sensor: GPU lidar publishing on a gz transport topic -->
- <gazebo reference="laser_frame">
+  <gazebo reference="laser_frame">
         <material>Gazebo/Black</material>
         <sensor name="laser" type="gpu_lidar">

Commit message: 

File: description/lidar.xacro (robot description, xacro)
@@ -1,38 +1,46 @@
 <?xml version="1.0"?>
 <robot xmlns:xacro="http://www.ros.org/wiki/xacro" >
-    <!-- ========= LiDAR "inside chassis" with an optical frame above top ======== -->
-  <!-- ===== LiDAR mount (centered above the chassis) ===== -->
-  <!-- LiDAR puck body -->
-  <link name="laser_frame">
+  <!-- ========= LiDAR "inside chassis" with an optical frame above top ======== -->
+  <!-- 1) A hidden LiDAR body inside the chassis (visual only, tiny collision) -->
+  <link name="lidar_body">
     <visual>
-      <origin xyz="0 0 0" rpy="0 0 0"/>
-      <geometry><cylinder radius="0.05" length="0.04"/></geometry>
-      <material name="black"/>
-    </visual>
-    <!-- little mast (optional visual) -->
-    <visual>
-      <origin xyz="0 0 -0.05" rpy="0 0 0"/>
-      <geometry><cylinder radius="0.01" length="0.10"/></geometry>
-      <material name="black"/>
+      <!-- Put the can inside the 10 mm-thick chassis plate -->
+      <!-- chassis center is at z=0.02, thickness=0.01 -> top at 0.025 -->
+      <origin xyz="0 0 0.02" rpy="0 0 0"/>
+      <geometry>
+        <cylinder radius="0.025" length="0.03"/>
+      </geometry>
+      <material name="blue"/>
     </visual>
     <collision>
-      <origin xyz="0 0 0" rpy="0 0 0"/>
-      <geometry><cylinder radius="0.05" length="0.04"/></geometry>
+      <!-- Tiny collision so it doesn't interfere with rays -->
+      <origin xyz="0 0 0.02" rpy="0 0 0"/>
+      <geometry>
+        <sphere radius="0.001"/>
+      </geometry>
     </collision>
-    <!-- simple inertial; adjust if needed -->
     <inertial>
-      <origin xyz="0 0 0" rpy="0 0 0"/>
-      <mass value="0.10"/>
-      <inertia ixx="1.0e-4" ixy="0" ixz="0" iyy="1.0e-4" iyz="0" izz="2.0e-4"/>
+      <origin xyz="0 0 0.02" rpy="0 0 0"/>
+      <mass value="0.15"/>
+      <inertia ixx="1e-4" ixy="0" ixz="0" iyy="1e-4" iyz="0" izz="1e-4"/>
     </inertial>
   </link>
-  <!-- Fixed mount: centered in XY, raised in Z (6 cm above chassis top) -->
-  <joint name="joint-chassis-lidar" type="fixed">
+  <!-- Fixed mount: lidar_body is bolted to the chassis center -->
+  <joint name="joint-chassis-lidar_body" type="fixed">
     <parent link="chassis-link"/>
-    <child link="laser_frame"/>
-    <origin xyz="0 0 0.06" rpy="0 0 0"/>
+    <child  link="lidar_body"/>
+    <origin xyz="0 0 0" rpy="0 0 0"/>
+  </joint>
+  <!-- 2) The optical frame (where the scan originates) just above the chassis top -->
+  <link name="laser_frame"/>
+  <joint name="joint-lidar_body-laser_frame" type="fixed">
+    <parent link="lidar_body"/>
+    <!-- Place the optical frame slightly above the top surface to avoid self-hits -->
+    <!-- chassis top = 0.025; put optical frame at 0.028 (3 mm clearance) -->
+    <child  link="laser_frame"/>
+    <origin xyz="0 0 0.001" rpy="0 0 0"/>
   </joint>
   <!-- Gazebo Fortress (gz-sim) sensor: GPU lidar publishing on a gz transport topic -->
-  <gazebo reference="laser_frame">
+ <gazebo reference="laser_frame">
         <material>Gazebo/Black</material>
         <sensor name="laser" type="gpu_lidar">

Commit message: 

File: description/lidar.xacro (robot description, xacro)
@@ -1,43 +1,25 @@
 <?xml version="1.0"?>
 <robot xmlns:xacro="http://www.ros.org/wiki/xacro" >
-  <!-- ========= LiDAR "inside chassis" with an optical frame above top ======== -->
-  <!-- 1) A hidden LiDAR body inside the chassis (visual only, tiny collision) -->
-  <link name="lidar_body">
+  <!-- LiDAR link (puck) -->
+  <link name="laser_frame">
     <visual>
-      <!-- Put the can inside the 10 mm-thick chassis plate -->
-      <!-- chassis center is at z=0.02, thickness=0.01 -> top at 0.025 -->
-      <origin xyz="0 0 0.02" rpy="0 0 0"/>
-      <geometry>
-        <cylinder radius="0.025" length="0.03"/>
-      </geometry>
-      <material name="blue"/>
+      <origin xyz="0 0 0" rpy="0 0 0"/>
+      <geometry><cylinder radius="0.05" length="0.04"/></geometry>
     </visual>
     <collision>
-      <!-- Tiny collision so it doesn't interfere with rays -->
-      <origin xyz="0 0 0.02" rpy="0 0 0"/>
-      <geometry>
-        <sphere radius="0.001"/>
-      </geometry>
+      <origin xyz="0 0 0" rpy="0 0 0"/>
+      <geometry><cylinder radius="0.05" length="0.04"/></geometry>
     </collision>
     <inertial>
-      <origin xyz="0 0 0.02" rpy="0 0 0"/>
-      <mass value="0.15"/>
-      <inertia ixx="1e-4" ixy="0" ixz="0" iyy="1e-4" iyz="0" izz="1e-4"/>
+      <origin xyz="0 0 0" rpy="0 0 0"/>
+      <mass value="0.10"/>
+      <inertia ixx="1e-4" ixy="0" ixz="0" iyy="1e-4" iyz="0" izz="2e-4"/>
     </inertial>
   </link>
-  <!-- Fixed mount: lidar_body is bolted to the chassis center -->
-  <joint name="joint-chassis-lidar_body" type="fixed">
-    <parent link="chassis-link"/>
-    <child  link="lidar_body"/>
-    <origin xyz="0 0 0" rpy="0 0 0"/>
-  </joint>
-  <!-- 2) The optical frame (where the scan originates) just above the chassis top -->
-  <link name="laser_frame"/>
-  <joint name="joint-lidar_body-laser_frame" type="fixed">
-    <parent link="lidar_body"/>
-    <!-- Place the optical frame slightly above the top surface to avoid self-hits -->
-    <!-- chassis top = 0.025; put optical frame at 0.028 (3 mm clearance) -->
-    <child  link="laser_frame"/>
-    <origin xyz="0 0 0.001" rpy="0 0 0"/>
+  <!-- Fixed mount: center of chassis, 6 cm up (adjust if you want) -->
+  <joint name="joint-chassis-lidar" type="fixed">
+    <parent link="chassis-link"/>       <!-- change to "chassis" if that's your name -->
+    <child link="laser_frame"/>
+    <origin xyz="0 0 0.06" rpy="0 0 0"/>
   </joint>
   <!-- Gazebo Fortress (gz-sim) sensor: GPU lidar publishing on a gz transport topic -->

Commit message: 

File: description/lidar.xacro (robot description, xacro)
@@ -1,23 +1,32 @@
 <?xml version="1.0"?>
 <robot xmlns:xacro="http://www.ros.org/wiki/xacro" >
-  <!-- LiDAR link (puck) -->
+  <!-- === Tiny LiDAR puck (visual only) === -->
   <link name="laser_frame">
+    <!-- Small top puck: radius 0.015 m, height 0.015 m -->
     <visual>
       <origin xyz="0 0 0" rpy="0 0 0"/>
-      <geometry><cylinder radius="0.05" length="0.04"/></geometry>
+      <geometry><cylinder radius="0.015" length="0.015"/></geometry>
+      <material name="blue"/>
+    </visual>
+    <!-- Optional skinny mast so it looks mounted -->
+    <visual>
+      <origin xyz="0 0 -0.02" rpy="0 0 0"/>
+      <geometry><cylinder radius="0.004" length="0.04"/></geometry>
+      <material name="blue"/>
     </visual>
     <collision>
       <origin xyz="0 0 0" rpy="0 0 0"/>
-      <geometry><cylinder radius="0.05" length="0.04"/></geometry>
+      <geometry><cylinder radius="0.015" length="0.015"/></geometry>
     </collision>
+    <!-- Light inertial to match the tiny visual -->
     <inertial>
       <origin xyz="0 0 0" rpy="0 0 0"/>
-      <mass value="0.10"/>
-      <inertia ixx="1e-4" ixy="0" ixz="0" iyy="1e-4" iyz="0" izz="2e-4"/>
+      <mass value="0.05"/>
+      <inertia ixx="5e-5" ixy="0" ixz="0" iyy="5e-5" iyz="0" izz="8e-5"/>
     </inertial>
   </link>
-  <!-- Fixed mount: center of chassis, 6 cm up (adjust if you want) -->
+  <!-- Fixed mount: centered on chassis, ~6 cm above it (adjust as you like) -->
   <joint name="joint-chassis-lidar" type="fixed">
-    <parent link="chassis-link"/>       <!-- change to "chassis" if that's your name -->
+    <parent link="chassis-link"/>
     <child link="laser_frame"/>
     <origin xyz="0 0 0.06" rpy="0 0 0"/>

Commit message: 

File: description/lidar.xacro (robot description, xacro)
@@ -1,34 +1,43 @@
 <?xml version="1.0"?>
 <robot xmlns:xacro="http://www.ros.org/wiki/xacro" >
-  <!-- === Tiny LiDAR puck (visual only) === -->
-  <link name="laser_frame">
-    <!-- Small top puck: radius 0.015 m, height 0.015 m -->
+  <!-- ========= LiDAR "inside chassis" with an optical frame above top ======== -->
+  <!-- 1) A hidden LiDAR body inside the chassis (visual only, tiny collision) -->
+  <link name="lidar_body">
     <visual>
-      <origin xyz="0 0 0" rpy="0 0 0"/>
-      <geometry><cylinder radius="0.015" length="0.015"/></geometry>
-      <material name="blue"/>
-    </visual>
-    <!-- Optional skinny mast so it looks mounted -->
-    <visual>
-      <origin xyz="0 0 -0.02" rpy="0 0 0"/>
-      <geometry><cylinder radius="0.004" length="0.04"/></geometry>
+      <!-- Put the can inside the 10 mm-thick chassis plate -->
+      <!-- chassis center is at z=0.02, thickness=0.01 -> top at 0.025 -->
+      <origin xyz="0 0 0.02" rpy="0 0 0"/>
+      <geometry>
+        <cylinder radius="0.025" length="0.03"/>
+      </geometry>
       <material name="blue"/>
     </visual>
     <collision>
-      <origin xyz="0 0 0" rpy="0 0 0"/>
-      <geometry><cylinder radius="0.015" length="0.015"/></geometry>
+      <!-- Tiny collision so it doesn't interfere with rays -->
+      <origin xyz="0 0 0.02" rpy="0 0 0"/>
+      <geometry>
+        <sphere radius="0.001"/>
+      </geometry>
     </collision>
-    <!-- Light inertial to match the tiny visual -->
     <inertial>
-      <origin xyz="0 0 0" rpy="0 0 0"/>
-      <mass value="0.05"/>
-      <inertia ixx="5e-5" ixy="0" ixz="0" iyy="5e-5" iyz="0" izz="8e-5"/>
+      <origin xyz="0 0 0.02" rpy="0 0 0"/>
+      <mass value="0.15"/>
+      <inertia ixx="1e-4" ixy="0" ixz="0" iyy="1e-4" iyz="0" izz="1e-4"/>
     </inertial>
   </link>
-  <!-- Fixed mount: centered on chassis, ~6 cm above it (adjust as you like) -->
-  <joint name="joint-chassis-lidar" type="fixed">
+  <!-- Fixed mount: lidar_body is bolted to the chassis center -->
+  <joint name="joint-chassis-lidar_body" type="fixed">
     <parent link="chassis-link"/>
-    <child link="laser_frame"/>
-    <origin xyz="0 0 0.06" rpy="0 0 0"/>
+    <child  link="lidar_body"/>
+    <origin xyz="0 0 0" rpy="0 0 0"/>
+  </joint>
+  <!-- 2) The optical frame (where the scan originates) just above the chassis top -->
+  <link name="laser_frame"/>
+  <joint name="joint-lidar_body-laser_frame" type="fixed">
+    <parent link="lidar_body"/>
+    <!-- Place the optical frame slightly above the top surface to avoid self-hits -->
+    <!-- chassis top = 0.025; put optical frame at 0.028 (3 mm clearance) -->
+    <child  link="laser_frame"/>
+    <origin xyz="0 0 0" rpy="0 0 0"/>
   </joint>
   <!-- Gazebo Fortress (gz-sim) sensor: GPU lidar publishing on a gz transport topic -->

Commit message: 

File: description/lidar.xacro (robot description, xacro)
@@ -1,43 +1,25 @@
 <?xml version="1.0"?>
 <robot xmlns:xacro="http://www.ros.org/wiki/xacro" >
-  <!-- ========= LiDAR "inside chassis" with an optical frame above top ======== -->
-  <!-- 1) A hidden LiDAR body inside the chassis (visual only, tiny collision) -->
-  <link name="lidar_body">
+  <!-- Tiny puck; no mast -->
+  <link name="laser_frame">
     <visual>
-      <!-- Put the can inside the 10 mm-thick chassis plate -->
-      <!-- chassis center is at z=0.02, thickness=0.01 -> top at 0.025 -->
-      <origin xyz="0 0 0.02" rpy="0 0 0"/>
-      <geometry>
-        <cylinder radius="0.025" length="0.03"/>
-      </geometry>
-      <material name="blue"/>
+      <origin xyz="0 0 0" rpy="0 0 0"/>
+      <geometry><cylinder radius="0.012" length="0.010"/></geometry>
     </visual>
     <collision>
-      <!-- Tiny collision so it doesn't interfere with rays -->
-      <origin xyz="0 0 0.02" rpy="0 0 0"/>
-      <geometry>
-        <sphere radius="0.001"/>
-      </geometry>
+      <!-- keep collision small too -->
+      <origin xyz="0 0 0" rpy="0 0 0"/>
+      <geometry><cylinder radius="0.012" length="0.010"/></geometry>
     </collision>
     <inertial>
-      <origin xyz="0 0 0.02" rpy="0 0 0"/>
-      <mass value="0.15"/>
-      <inertia ixx="1e-4" ixy="0" ixz="0" iyy="1e-4" iyz="0" izz="1e-4"/>
+      <mass value="0.03"/>
+      <inertia ixx="3e-5" ixy="0" ixz="0" iyy="3e-5" iyz="0" izz="5e-5"/>
     </inertial>
   </link>
-  <!-- Fixed mount: lidar_body is bolted to the chassis center -->
-  <joint name="joint-chassis-lidar_body" type="fixed">
+  <joint name="joint-chassis-lidar" type="fixed">
     <parent link="chassis-link"/>
-    <child  link="lidar_body"/>
-    <origin xyz="0 0 0" rpy="0 0 0"/>
-  </joint>
-  <!-- 2) The optical frame (where the scan originates) just above the chassis top -->
-  <link name="laser_frame"/>
-  <joint name="joint-lidar_body-laser_frame" type="fixed">
-    <parent link="lidar_body"/>
-    <!-- Place the optical frame slightly above the top surface to avoid self-hits -->
-    <!-- chassis top = 0.025; put optical frame at 0.028 (3 mm clearance) -->
-    <child  link="laser_frame"/>
-    <origin xyz="0 0 0" rpy="0 0 0"/>
+    <child link="laser_frame"/>
+    <!-- lift it a bit so it clears the deck -->
+    <origin xyz="0 0 0.08" rpy="0 0 0"/>
   </joint>
   <!-- Gazebo Fortress (gz-sim) sensor: GPU lidar publishing on a gz transport topic -->

Commit message: 

File: description/lidar.xacro (robot description, xacro)
@@ -1,49 +1,51 @@
 <?xml version="1.0"?>
 <robot xmlns:xacro="http://www.ros.org/wiki/xacro" >
-  <!-- Tiny puck; no mast -->
-  <link name="laser_frame">
-    <visual>
-      <origin xyz="0 0 0" rpy="0 0 0"/>
-      <geometry><cylinder radius="0.012" length="0.010"/></geometry>
-    </visual>
-    <collision>
-      <!-- keep collision small too -->
-      <origin xyz="0 0 0" rpy="0 0 0"/>
-      <geometry><cylinder radius="0.012" length="0.010"/></geometry>
-    </collision>
-    <inertial>
-      <mass value="0.03"/>
-      <inertia ixx="3e-5" ixy="0" ixz="0" iyy="3e-5" iyz="0" izz="5e-5"/>
-    </inertial>
-  </link>
-  <joint name="joint-chassis-lidar" type="fixed">
-    <parent link="chassis-link"/>
-    <child link="laser_frame"/>
-    <!-- lift it a bit so it clears the deck -->
-    <origin xyz="0 0 0.08" rpy="0 0 0"/>
-  </joint>
-  <!-- Gazebo Fortress (gz-sim) sensor: GPU lidar publishing on a gz transport topic -->
- <gazebo reference="laser_frame">
-        <material>Gazebo/Black</material>
-        <sensor name="laser" type="gpu_lidar">
-            <pose> 0 0 0 0 0 0 </pose>
-            <visualize>false</visualize>
-            <update_rate>10</update_rate>
-            <lidar>
-                <scan>
-                    <horizontal>
-                        <samples>360</samples>
-                        <min_angle>-3.14</min_angle>
-                        <max_angle>3.14</max_angle>
-                    </horizontal>
-                </scan>
-                <range>
-                    <min>0.3</min>
-                    <max>12</max>
-                </range>
-            </lidar>
-            <topic>scan</topic>
-            <gz_frame_id>laser_frame</gz_frame_id>
-        </sensor>
-    </gazebo>
+  <!-- LiDAR puck mounted on TOP of the rear package box -->
+<link name="laser_frame">
+  <visual>
+    <origin xyz="0 0 0" rpy="0 0 0"/>
+    <geometry><cylinder radius="0.012" length="0.010"/></geometry>
+    <material name="black"><color rgba="0.05 0.05 0.05 1"/></material>
+  </visual>
+  <collision>
+    <origin xyz="0 0 0" rpy="0 0 0"/>
+    <geometry><cylinder radius="0.012" length="0.010"/></geometry>
+  </collision>
+  <inertial>
+    <mass value="0.03"/>
+    <inertia ixx="3e-5" ixy="0" ixz="0" iyy="3e-5" iyz="0" izz="5e-5"/>
+  </inertial>
+</link>
+<!-- IMPORTANT: parent is the package box, not the chassis -->
+<joint name="joint-chassis-lidar" type="fixed">
+  <parent link="package_box_link"/>
+  <child  link="laser_frame"/>
+  <!-- Centered on the box in X/Y; sits exactly on the top surface:
+       z_offset = 0.186/2 + 0.010/2 = 0.098 -->
+  <origin xyz="0 0 0.098" rpy="0 0 0"/>
+</joint>
+<!-- Gazebo sensor attached to the LiDAR link -->
+<gazebo reference="laser_frame">
+  <material>Gazebo/Black</material>
+  <sensor name="laser" type="gpu_lidar">
+    <pose>0 0 0 0 0 0</pose>
+    <visualize>false</visualize>
+    <update_rate>10</update_rate>
+    <lidar>
+      <scan>
+        <horizontal>
+          <samples>360</samples>
+          <min_angle>-3.14159</min_angle>
+          <max_angle> 3.14159</max_angle>
+        </horizontal>
+      </scan>
+      <range>
+        <min>0.3</min>
+        <max>12.0</max>
+      </range>
+    </lidar>
+    <topic>scan</topic>
+    <gz_frame_id>laser_frame</gz_frame_id>
+  </sensor>
+</gazebo>
 </robot>

File: description/robot.urdf.xacro (robot description, xacro)
@@ -5,3 +5,4 @@
     <xacro:include filename="robot_core.xacro" />
     <xacro:include filename="ros2_control.xacro" />
+    <xacro:include filename="lidar.xacro" />
 </robot>
