Commit message: 

File: description/robot_core.xacro (robot description, xacro)
@@ -1,22 +1,20 @@
 <?xml version="1.0"?>
 <robot xmlns:xacro="http://www.ros.org/wiki/xacro" >
-  <!-- BASE LINK -->
-  <link name="base_link">
-  </link>
-  <!-- BASE_FOOTPRINT LINK -->
+  <!-- ===== BASE LINK ===== -->
+  <link name="base_link"/>
+  <!-- base_footprint -->
   <joint name="base_footprint_joint" type="fixed">
-      <parent link="base_link"/>
-      <child link="base_footprint"/>
-      <origin xyz="0 0 0" rpy="0 0 0"/>
+    <parent link="base_link"/>
+    <child  link="base_footprint"/>
+    <origin xyz="0 0 0" rpy="0 0 0"/>
   </joint>
-  <link name="base_footprint">
-  </link>
-  <!--chassis link-->
+  <link name="base_footprint"/>
+  <!-- ===== CHASSIS ===== -->
+  <!-- from UGV02 DXF top view: 252.336 x 239.796 x 10 mm -->
   <link name="chassis-link">
     <visual>
-      <origin rpy="0 0 0" xyz="0 0 0"/>
+      <origin xyz="0 0 0" rpy="0 0 0"/>
       <geometry>
-        <!-- from PDF: ~120.02 x 112.87 x 10 mm -->
-        <box size="0.12002 0.11287 0.01"/>
+        <box size="0.252336 0.239796 0.01"/>
       </geometry>
       <material name="brown">
@@ -25,156 +23,176 @@
     </visual>
     <collision>
-      <origin rpy="0 0 0" xyz="0 0 0"/>
+      <origin xyz="0 0 0" rpy="0 0 0"/>
       <geometry>
-        <box size="0.12002 0.11287 0.01"/>
+        <box size="0.252336 0.239796 0.01"/>
       </geometry>
     </collision>
     <inertial>
+      <!-- you can tune mass later if you have a measured value -->
       <mass value="0.6"/>
-      <!-- box inertia about its center: ixx=m*(y^2+z^2)/12 etc. -->
-      <inertia ixx="0.000641981845" ixy="0" ixz="0" iyy="0.00072524002" iyz="0" izz="0.001357221865"/>
+      <inertia ixx="0.00065" ixy="0" ixz="0" iyy="0.00073" iyz="0" izz="0.00136"/>
     </inertial>
   </link>
+  <!-- original vertical offset kept -->
   <joint name="joint-base-chassis" type="fixed">
     <parent link="base_link"/>
-    <child link="chassis-link"/>
-    <!-- keep same height reference as your original (raise chassis center 20 mm) -->
-    <origin rpy="0 0 0" xyz="0 0 0.02"/>
+    <child  link="chassis-link"/>
+    <origin xyz="0 0 0.02" rpy="0 0 0"/>
   </joint>
   <material name="blue">
     <color rgba="0 0.4 0.5 1"/>
   </material>
-  <!-- ${x_position}-${y_position}-wheel-link -->
+  <!-- ===== WHEEL TEMPLATE (values inlined for clarity) =====
+       wheel radius from DXF arcs ~39.65 mm -> radius="0.03965"
+       wheel length (tread width) assumed 0.04 m (adjust if you know exact)
+  -->
+  <!-- ========== RIGHT SIDE (front, mid, rear) ========== -->
+  <!-- FRONT RIGHT (existing) -->
   <link name="front-right-wheel-link">
     <visual>
-      <origin rpy="1.5707963267948966 0 0" xyz="0 0 0"/>
-      <geometry>
-        <!-- from PDF: wheel Ø~58 mm, width ~12 mm -->
-        <cylinder length="0.012" radius="0.029"/>
-      </geometry>
+      <origin xyz="0 0 0" rpy="1.5707963267948966 0 0"/>
+      <geometry><cylinder length="0.04" radius="0.03965"/></geometry>
       <material name="blue"/>
     </visual>
     <collision>
-      <origin rpy="1.5707963267948966 0 0" xyz="0 0 0"/>
-      <geometry>
-        <cylinder length="0.012" radius="0.029"/>
-      </geometry>
+      <origin xyz="0 0 0" rpy="1.5707963267948966 0 0"/>
+      <geometry><cylinder length="0.04" radius="0.03965"/></geometry>
     </collision>
     <inertial>
-      <origin rpy="1.5707963267948966 0 0" xyz="0 0 0"/>
+      <origin xyz="0 0 0" rpy="1.5707963267948966 0 0"/>
       <mass value="0.15"/>
-      <inertia ixx="3.33375e-05" ixy="0" ixz="0" iyy="3.33375e-05" iyz="0" izz="6.3075e-05"/>
+      <inertia ixx="3.4e-05" ixy="0" ixz="0" iyy="3.4e-05" iyz="0" izz="6.3e-05"/>
     </inertial>
   </link>
   <joint name="joint-chassis-front-right-wheel" type="continuous">
     <parent link="chassis-link"/>
-    <child link="front-right-wheel-link"/>
-    <!-- place wheel centers near the corners using new chassis size -->
-    <origin rpy="0 0 0" xyz="0.03101 0.051435 0"/>
+    <child  link="front-right-wheel-link"/>
+    <origin xyz="0.086 0.105 0" rpy="0 0 0"/>
     <axis xyz="0 1 0"/>
   </joint>
-  <!-- ${x_position}-${y_position}-wheel-link -->
-  <link name="front-left-wheel-link">
+  <!-- MID RIGHT (NEW) -->
+  <link name="mid-right-wheel-link">
     <visual>
-      <origin rpy="1.5707963267948966 0 0" xyz="0 0 0"/>
-      <geometry>
-        <cylinder length="0.012" radius="0.029"/>
-      </geometry>
+      <origin xyz="0 0 0" rpy="1.5707963267948966 0 0"/>
+      <geometry><cylinder length="0.04" radius="0.03965"/></geometry>
       <material name="blue"/>
     </visual>
     <collision>
-      <origin rpy="1.5707963267948966 0 0" xyz="0 0 0"/>
-      <geometry>
-        <cylinder length="0.012" radius="0.029"/>
-      </geometry>
+      <origin xyz="0 0 0" rpy="1.5707963267948966 0 0"/>
+      <geometry><cylinder length="0.04" radius="0.03965"/></geometry>
     </collision>
     <inertial>
-      <origin rpy="1.5707963267948966 0 0" xyz="0 0 0"/>
+      <origin xyz="0 0 0" rpy="1.5707963267948966 0 0"/>
       <mass value="0.15"/>
-      <inertia ixx="3.33375e-05" ixy="0" ixz="0" iyy="3.33375e-05" iyz="0" izz="6.3075e-05"/>
+      <inertia ixx="3.4e-05" ixy="0" ixz="0" iyy="3.4e-05" iyz="0" izz="6.3e-05"/>
+    </inertial>
+  </link>
+  <joint name="joint-chassis-mid-right-wheel" type="continuous">
+    <parent link="chassis-link"/>
+    <child  link="mid-right-wheel-link"/>
+    <origin xyz="0.000 0.105 0" rpy="0 0 0"/>
+    <axis xyz="0 1 0"/>
+  </joint>
+  <!-- REAR RIGHT (existing “rare-right-wheel-link”) -->
+  <link name="rare-right-wheel-link">
+    <visual>
+      <origin xyz="0 0 0" rpy="1.5707963267948966 0 0"/>
+      <geometry><cylinder length="0.04" radius="0.03965"/></geometry>
+      <material name="blue"/>
+    </visual>
+    <collision>
+      <origin xyz="0 0 0" rpy="1.5707963267948966 0 0"/>
+      <geometry><cylinder length="0.04" radius="0.03965"/></geometry>
+    </collision>
+    <inertial>
+      <origin xyz="0 0 0" rpy="1.5707963267948966 0 0"/>
+      <mass value="0.15"/>
+      <inertia ixx="3.4e-05" ixy="0" ixz="0" iyy="3.4e-05" iyz="0" izz="6.3e-05"/>
+    </inertial>
+  </link>
+  <joint name="joint-chassis-rare-right-wheel" type="continuous">
+    <parent link="chassis-link"/>
+    <child  link="rare-right-wheel-link"/>
+    <origin xyz="-0.086 0.105 0" rpy="0 0 0"/>
+    <axis xyz="0 1 0"/>
+  </joint>
+  <!-- ========== LEFT SIDE (front, mid, rear) ========== -->
+  <!-- FRONT LEFT (existing) -->
+  <link name="front-left-wheel-link">
+    <visual>
+      <origin xyz="0 0 0" rpy="1.5707963267948966 0 0"/>
+      <geometry><cylinder length="0.04" radius="0.03965"/></geometry>
+      <material name="blue"/>
+    </visual>
+    <collision>
+      <origin xyz="0 0 0" rpy="1.5707963267948966 0 0"/>
+      <geometry><cylinder length="0.04" radius="0.03965"/></geometry>
+    </collision>
+    <inertial>
+      <origin xyz="0 0 0" rpy="1.5707963267948966 0 0"/>
+      <mass value="0.15"/>
+      <inertia ixx="3.4e-05" ixy="0" ixz="0" iyy="3.4e-05" iyz="0" izz="6.3e-05"/>
     </inertial>
   </link>
   <joint name="joint-chassis-front-left-wheel" type="continuous">
     <parent link="chassis-link"/>
-    <child link="front-left-wheel-link"/>
-    <origin rpy="0 0 0" xyz="0.03101 -0.051435 0"/>
+    <child  link="front-left-wheel-link"/>
+    <origin xyz="0.086 -0.105 0" rpy="0 0 0"/>
     <axis xyz="0 1 0"/>
   </joint>
-  <!-- ${x_position}-${y_position}-wheel-link -->
-  <link name="rare-right-wheel-link">
+  <!-- MID LEFT (NEW) -->
+  <link name="mid-left-wheel-link">
     <visual>
-      <origin rpy="1.5707963267948966 0 0" xyz="0 0 0"/>
-      <geometry>
-        <cylinder length="0.012" radius="0.029"/>
-      </geometry>
+      <origin xyz="0 0 0" rpy="1.5707963267948966 0 0"/>
+      <geometry><cylinder length="0.04" radius="0.03965"/></geometry>
       <material name="blue"/>
     </visual>
     <collision>
-      <origin rpy="1.5707963267948966 0 0" xyz="0 0 0"/>
-      <geometry>
-        <cylinder length="0.012" radius="0.029"/>
-      </geometry>
+      <origin xyz="0 0 0" rpy="1.5707963267948966 0 0"/>
+      <geometry><cylinder length="0.04" radius="0.03965"/></geometry>
     </collision>
     <inertial>
-      <origin rpy="1.5707963267948966 0 0" xyz="0 0 0"/>
+      <origin xyz="0 0 0" rpy="1.5707963267948966 0 0"/>
       <mass value="0.15"/>
-      <inertia ixx="3.33375e-05" ixy="0" ixz="0" iyy="3.33375e-05" iyz="0" izz="6.3075e-05"/>
+      <inertia ixx="3.4e-05" ixy="0" ixz="0" iyy="3.4e-05" iyz="0" izz="6.3e-05"/>
     </inertial>
   </link>
-  <joint name="joint-chassis-rare-right-wheel" type="continuous">
+  <joint name="joint-chassis-mid-left-wheel" type="continuous">
     <parent link="chassis-link"/>
-    <child link="rare-right-wheel-link"/>
-    <origin rpy="0 0 0" xyz="-0.03101 0.051435 0"/>
+    <child  link="mid-left-wheel-link"/>
+    <origin xyz="0.000 -0.105 0" rpy="0 0 0"/>
     <axis xyz="0 1 0"/>
   </joint>
-  <!-- ${x_position}-${y_position}-wheel-link -->
+  <!-- REAR LEFT (existing “rare-left-wheel-link”) -->
   <link name="rare-left-wheel-link">
     <visual>
-      <origin rpy="1.5707963267948966 0 0" xyz="0 0 0"/>
-      <geometry>
-        <cylinder length="0.012" radius="0.029"/>
-      </geometry>
-      <material name="blue"/>
+      <origin xyz="0 0 0" rpy="1.5707963267948966 0 0"/>
+      <geometry><cylinder length="0.04" radius="0.03965"/></geometry>
     </visual>
     <collision>
-      <origin rpy="1.5707963267948966 0 0" xyz="0 0 0"/>
-      <geometry>
-        <cylinder length="0.012" radius="0.029"/>
-      </geometry>
+      <origin xyz="0 0 0" rpy="1.5707963267948966 0 0"/>
+      <geometry><cylinder length="0.04" radius="0.03965"/></geometry>
     </collision>
     <inertial>
-      <origin rpy="1.5707963267948966 0 0" xyz="0 0 0"/>
+      <origin xyz="0 0 0" rpy="1.5707963267948966 0 0"/>
       <mass value="0.15"/>
-      <inertia ixx="3.33375e-05" ixy="0" ixz="0" iyy="3.33375e-05" iyz="0" izz="6.3075e-05"/>
+      <inertia ixx="3.4e-05" ixy="0" ixz="0" iyy="3.4e-05" iyz="0" izz="6.3e-05"/>
     </inertial>
   </link>
   <joint name="joint-chassis-rare-left-wheel" type="continuous">
     <parent link="chassis-link"/>
-    <child link="rare-left-wheel-link"/>
-    <origin rpy="0 0 0" xyz="-0.03101 -0.051435 0"/>
+    <child  link="rare-left-wheel-link"/>
+    <origin xyz="-0.086 -0.105 0" rpy="0 0 0"/>
     <axis xyz="0 1 0"/>
   </joint>
+  <!-- ===== Gazebo material/friction (kept & extended) ===== -->
   <gazebo reference="chassis-link">
     <material>Gazebo/DarkGrey</material>
   </gazebo>
-  <gazebo reference="front-right-wheel-link">
-    <mu1>10000.0 </mu1>
-    <mu2>10000.0 </mu2>
-    <material>Gazebo/Purple</material>
-  </gazebo>
-  <gazebo reference="front-left-wheel-link">
-    <mu1>10000.0 </mu1>
-    <mu2>10000.0 </mu2>
-    <material>Gazebo/Purple</material>
-  </gazebo>
-  <gazebo reference="rare-right-wheel-link">
-    <mu1>10000.0 </mu1>
-    <mu2>10000.0 </mu2>
-    <material>Gazebo/Purple</material>
-  </gazebo>
-  <gazebo reference="rare-left-wheel-link">
-    <mu1>10000.0 </mu1>
-    <mu2>10000.0 </mu2>
-    <material>Gazebo/Purple</material>
-  </gazebo>
+  <gazebo reference="front-right-wheel-link"><mu1>10000.0</mu1><mu2>10000.0</mu2><material>Gazebo/Purple</material></gazebo>
+  <gazebo reference="mid-right-wheel-link"><mu1>10000.0</mu1><mu2>10000.0</mu2><material>Gazebo/Purple</material></gazebo>
+  <gazebo reference="rare-right-wheel-link"><mu1>10000.0</mu1><mu2>10000.0</mu2><material>Gazebo/Purple</material></gazebo>
+  <gazebo reference="front-left-wheel-link"><mu1>10000.0</mu1><mu2>10000.0</mu2><material>Gazebo/Purple</material></gazebo>
+  <gazebo reference="mid-left-wheel-link"><mu1>10000.0</mu1><mu2>10000.0</mu2><material>Gazebo/Purple</material></gazebo>
+  <gazebo reference="rare-left-wheel-link"><mu1>10000.0</mu1><mu2>10000.0</mu2><material>Gazebo/Purple</material></gazebo>
 </robot>

Commit message: 

File: description/robot_core.xacro (robot description, xacro)
@@ -196,3 +196,46 @@
   <gazebo reference="mid-left-wheel-link"><mu1>10000.0</mu1><mu2>10000.0</mu2><material>Gazebo/Purple</material></gazebo>
   <gazebo reference="rare-left-wheel-link"><mu1>10000.0</mu1><mu2>10000.0</mu2><material>Gazebo/Purple</material></gazebo>
+<!-- ===== Package box (rear cargo) =====
+     Dimensions (mm): width=200, height=186, depth(extrude)=100
+     URDF (m): X=0.10, Y=0.20, Z=0.186
+-->
+<link name="package_box_link">
+  <visual>
+    <origin xyz="0 0 0" rpy="0 0 0"/>
+    <geometry>
+      <box size="0.10 0.20 0.186"/>
+    </geometry>
+    <material name="cargo_purple">
+      <color rgba="0.6 0.2 0.8 1"/>
+    </material>
+  </visual>
+  <collision>
+    <origin xyz="0 0 0" rpy="0 0 0"/>
+    <geometry>
+      <box size="0.10 0.20 0.186"/>
+    </geometry>
+  </collision>
+  <inertial>
+    <origin xyz="0 0 0" rpy="0 0 0"/>
+    <mass value="0.5"/>
+    <inertia ixx="0.003108" ixy="0" ixz="0"
+             iyy="0.001858" iyz="0"
+             izz="0.002083"/>
+  </inertial>
+</link>
+<joint name="joint-chassis-package-box" type="fixed">
+  <parent link="chassis-link"/>
+  <child  link="package_box_link"/>
+  <!-- Place at rear (−X), centered in Y, sitting on chassis top -->
+  <!-- chassis: 0.252336 x 0.239796 x 0.01 -->
+  <origin xyz="-0.0712 0 0.02" rpy="0 0 0"/>
+</joint>
+<!-- ===== Gazebo visualization & physics ===== -->
+<gazebo reference="package_box_link">
+  <material>Gazebo/Yellow</material>
+  <mu1>1.0</mu1>       <!-- friction coefficient 1 -->
+  <mu2>1.0</mu2>       <!-- friction coefficient 2 -->
+  <kp>100000.0</kp>    <!-- contact stiffness -->
+  <kd>1.0</kd>         <!-- damping -->
+</gazebo>
 </robot>

Commit message: 

File: description/robot_core.xacro (robot description, xacro)
@@ -229,5 +229,5 @@
   <!-- Place at rear (−X), centered in Y, sitting on chassis top -->
   <!-- chassis: 0.252336 x 0.239796 x 0.01 -->
-  <origin xyz="-0.0712 0 0.02" rpy="0 0 0"/>
+  <origin xyz="-0.0712 0 0.098" rpy="0 0 0"/>
 </joint>
 <!-- ===== Gazebo visualization & physics ===== -->

Commit message: 

File: description/robot_core.xacro (robot description, xacro)
@@ -88,4 +88,5 @@
     </inertial>
   </link>
+  <!-- MID RIGHT (free-rolling, mimics front-right) -->
   <joint name="joint-chassis-mid-right-wheel" type="continuous">
     <parent link="chassis-link"/>
@@ -93,4 +94,6 @@
     <origin xyz="0.000 0.105 0" rpy="0 0 0"/>
     <axis xyz="0 1 0"/>
+    <!-- make the mid wheel spin exactly like the powered right wheel -->
+    <mimic joint="joint-chassis-front-right-wheel" multiplier="1.0" offset="0.0"/>
   </joint>
   <!-- REAR RIGHT (existing “rare-right-wheel-link”) -->
@@ -158,4 +161,5 @@
     </inertial>
   </link>
+  <!-- MID LEFT (free-rolling, mimics front-left) -->
   <joint name="joint-chassis-mid-left-wheel" type="continuous">
     <parent link="chassis-link"/>
@@ -163,4 +167,6 @@
     <origin xyz="0.000 -0.105 0" rpy="0 0 0"/>
     <axis xyz="0 1 0"/>
+    <!-- make the mid wheel spin exactly like the powered left wheel -->
+    <mimic joint="joint-chassis-front-left-wheel" multiplier="1.0" offset="0.0"/>
   </joint>
   <!-- REAR LEFT (existing “rare-left-wheel-link”) -->
